File: RC-Car-Project/Xbee_sch.kicad_sch (KiCad schematic)
At the start: 0 parts

Commit message: XBEE + connector and mcu connector
Parts:
- added U1: XBee_SMT, RF_Module:Digi_XBee_SMT, symbol RF_ZigBee:XBee_SMT
Connections:
- new net +3V3: U1.2 (VCC)
- new net GND_3V3: U1.1 (GND), U1.11 (GND), U1.13 (GND), U1.22 (GND), U1.27 (VREF), U1.35 (GND)
- new net UART_RX: U1.4 (DIO14/UART_RX/~{CONFIG})
- new net UART_TX: U1.3 (DIO13/UART_TX)
Other:
- note added: "XBEE Zigbee User Guide: https://www.digi.com/resources/documentation/digidocs/pdfs/90000976.pdf"

Commit message: Add libraries and components in schs
Parts:
- removed U1: XBee_SMT, RF_Module:Digi_XBee_SMT, symbol RF_ZigBee:XBee_SMT
Other:
- note removed: "XBEE Zigbee User Guide: https://www.digi.com/resources/documentation/digidocs/pdfs/90000976.pdf"
