File: RC-Car-Project/_autosave-IVTSense.kicad_sch (KiCad schematic)
At the start: 12 parts, among them U7 INA229AQDGSRQ1, U8 ADC082S021CIMM/NOPB

Commit message: Added Fuze
Parts:
- F1: footprint FUS_SF-3812F_BRN -> SF-3812F6000T-2:FUS_SF-3812F_BRN
Changed lines of the file:
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@@
 			)
 		)
-		(property "Footprint" "FUS_SF-3812F_BRN"
+		(property "Footprint" "SF-3812F6000T-2:FUS_SF-3812F_BRN"
 			(at 195.58 105.41 0)
 			(effects
