File: RC-Car-Project/RF_sch.kicad_sch (KiCad schematic)
At the start: 35 parts

Commit message: Add caps
Parts:
- C18, C33: MANUF_PN (none) -> CL10A106KP8NNNC
- C19, C31, C35: value 100nF/10V -> 0.1uF/10V; MANUF_PN (none) -> C0603C104K5RAC7411
- C32, C34: now not fitted
Changed lines of the file:
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@@
 		(in_bom yes)
 		(on_board yes)
-		(dnp no)
+		(dnp yes)
 		(property "Reference" "C34"
 			(at 179.07 81.28 0)
@@
 			)
 		)
-		(property "Value" "100nF/10V"
+		(property "Value" "0.1uF/10V"
 			(at 187.706 58.674 0)
 			(effects
@@
 			)
 		)
-		(property "MANUF_PN" ""
+		(property "MANUF_PN" "C0603C104K5RAC7411"
 			(at 186.69 55.88 0)
 			(effects
@@
 			)
 		)
-		(property "MANUF_PN" ""
+		(property "MANUF_PN" "CL10A106KP8NNNC"
 			(at 175.26 55.88 0)
 			(effects
@@
 			)
 		)
-		(property "Value" "100nF/10V"
+		(property "Value" "0.1uF/10V"
 			(at 155.956 58.674 0)
 			(effects
@@
 			)
 		)
-		(property "MANUF_PN" ""
+		(property "MANUF_PN" "C0603C104K5RAC7411"
 			(at 154.94 55.88 0)
 			(effects
@@
 			)
 		)
-		(property "MANUF_PN" ""
+		(property "MANUF_PN" "CL10A106KP8NNNC"
 			(at 128.27 55.88 0)
 			(effects
@@
 		(in_bom yes)
 		(on_board yes)
-		(dnp no)
+		(dnp yes)
 		(property "Reference" "C32"
 			(at 166.624 81.534 0)
@@
 			)
 		)
-		(property "Value" "100nF/10V"
+		(property "Value" "0.1uF/10V"
 			(at 140.716 58.674 0)
 			(effects
@@
 			)
 		)
-		(property "MANUF_PN" ""
+		(property "MANUF_PN" "C0603C104K5RAC7411"
 			(at 139.7 55.88 0)
 			(effects
