File: RC-Car-Project/RF_sch.kicad_sch (KiCad schematic)
At the start: 35 parts

Commit message: Fixed (AGAIN AGAIN)
Parts:
- renumbered C18 to C31, C19 to C32, C31 to C33, C32 to C34, C33 to C35, C34 to C36, C35 to C37, D6 to D10, D7 to D11, D5 to D9, R11 to R18, R12 to R19, R13 to R20, R34 to R21, R35 to R22, R36 to R23, R37 to R24, R38 to R25, R39 to R26, R40 to R27, R41 to R28, R42 to R29, R43 to R30, R44 to R31, R45 to R32, R46 to R33, R47 to R34, R48 to R35, R49 to R36, R50 to R37, R51 to R38, R63 to R39, R52 to R40, U2 to U5

Commit message: Add NA
Parts:
- C34, C36, D10, D11, D9: MANUF_PN (none) -> N/A
Changed lines of the file:
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@@
 			)
 		)
-		(property "MANUF_PN" ""
+		(property "MANUF_PN" "N/A"
 			(at 176.53 81.28 0)
 			(effects
@@
 			)
 		)
-		(property "MANUF_PN" ""
+		(property "MANUF_PN" "N/A"
 			(at 115.57 55.88 0)
 			(effects
@@
 			)
 		)
-		(property "MANUF_PN" ""
+		(property "MANUF_PN" "N/A"
 			(at 107.95 55.88 0)
 			(effects
@@
 			)
 		)
-		(property "MANUF_PN" ""
+		(property "MANUF_PN" "N/A"
 			(at 163.83 81.28 0)
 			(effects
@@
 			)
 		)
-		(property "MANUF_PN" ""
+		(property "MANUF_PN" "N/A"
 			(at 111.76 55.88 0)
 			(effects
