File: RC-Car-Project/MiscDriver.kicad_sch (KiCad schematic)
At the start: 12 parts, among them Q5 PMF250XNE, Q6 PMF250XNE, Q8 PMF250XNE, Q9 PMF250XNE

Commit message: Resistor manuf PNs labelled
resistor manufacturer part numbers added
Parts:
- R30, R31, R56, R57: MANUF_PN (none) -> RC0603FR-07100RL
- R32, R33, R58, R59: MANUF_PN (none) -> RC0603FR-0710KL
Changed lines of the file:
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@@
 			)
 		)
-		(property "MANUF_PN" ""
+		(property "MANUF_PN" "RC0603FR-07100RL"
 			(at 179.07 99.06 0)
 			(effects
@@
 			)
 		)
-		(property "MANUF_PN" ""
+		(property "MANUF_PN" "RC0603FR-07100RL"
 			(at 120.65 66.04 0)
 			(effects
@@
 			)
 		)
-		(property "MANUF_PN" ""
+		(property "MANUF_PN" "RC0603FR-0710KL"
 			(at 127 102.87 0)
 			(effects
@@
 			)
 		)
-		(property "MANUF_PN" ""
+		(property "MANUF_PN" "RC0603FR-07100RL"
 			(at 120.65 99.06 0)
 			(effects
@@
 			)
 		)
-		(property "MANUF_PN" ""
+		(property "MANUF_PN" "RC0603FR-07100RL"
 			(at 179.07 66.04 0)
 			(effects
@@
 			)
 		)
-		(property "MANUF_PN" ""
+		(property "MANUF_PN" "RC0603FR-0710KL"
 			(at 127 69.85 0)
 			(effects
@@
 			)
 		)
-		(property "MANUF_PN" ""
+		(property "MANUF_PN" "RC0603FR-0710KL"
 			(at 185.42 69.85 0)
 			(effects
@@
 			)
 		)
-		(property "MANUF_PN" ""
+		(property "MANUF_PN" "RC0603FR-0710KL"
 			(at 185.42 102.87 0)
 			(effects

Commit message: Fixed (AGAIN AGAIN)
Parts:
- renumbered Q5 to Q6, Q6 to Q7, R30 to R65, R31 to R66, R32 to R67, R33 to R68, R56 to R69, R57 to R70, R58 to R71, R59 to R72
Changed lines of the file:
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@@
 		(dnp no)
 		(fields_autoplaced yes)
-		(property "Reference" "R57"
+		(property "Reference" "R70"
 			(at 179.07 92.71 90)
 			(effects
@@
 			(project "RC-Car-Project"
 				(path "/ba870fd1-751d-4755-8e1a-1ea86ca9e2f6/6cd00c1a-14cd-4705-8fa1-76b1c50e2463"
-					(reference "R57")
+					(reference "R70")
 					(unit 1)
 				)
@@
 		(dnp no)
 		(fields_autoplaced yes)
-		(property "Reference" "#PWR0123"
+		(property "Reference" "#PWR0148"
 			(at 127 80.01 0)
 			(effects
@@
 			(project "RC-Car-Project"
 				(path "/ba870fd1-751d-4755-8e1a-1ea86ca9e2f6/6cd00c1a-14cd-4705-8fa1-76b1c50e2463"
-					(reference "#PWR0123")
+					(reference "#PWR0148")
 					(unit 1)
 				)
@@
 		(dnp no)
 		(fields_autoplaced yes)
-		(property "Reference" "#PWR0125"
+		(property "Reference" "#PWR0150"
 			(at 137.16 81.28 0)
 			(effects
@@
 			(project "RC-Car-Project"
 				(path "/ba870fd1-751d-4755-8e1a-1ea86ca9e2f6/6cd00c1a-14cd-4705-8fa1-76b1c50e2463"
-					(reference "#PWR0125")
+					(reference "#PWR0150")
 					(unit 1)
 				)
@@
 		(dnp no)
 		(fields_autoplaced yes)
-		(property "Reference" "R30"
+		(property "Reference" "R65"
 			(at 120.65 59.69 90)
 			(effects
@@
 			(project ""
 				(path "/ba870fd1-751d-4755-8e1a-1ea86ca9e2f6/6cd00c1a-14cd-4705-8fa1-76b1c50e2463"
-					(reference "R30")
+					(reference "R65")
 					(unit 1)
 				)
@@
 		(dnp no)
 		(fields_autoplaced yes)
-		(property "Reference" "R33"
+		(property "Reference" "R68"
 			(at 129.54 101.5999 0)
 			(effects
@@
 			(project "RC-Car-Project"
 				(path "/ba870fd1-751d-4755-8e1a-1ea86ca9e2f6/6cd00c1a-14cd-4705-8fa1-76b1c50e2463"
-					(reference "R33")
+					(reference "R68")
 					(unit 1)
 				)
@@
 		(dnp no)
 		(fields_autoplaced yes)
-		(property "Reference" "R31"
+		(property "Reference" "R66"
 			(at 120.65 92.71 90)
 			(effects
@@
 			(project "RC-Car-Project"
 				(path "/ba870fd1-751d-4755-8e1a-1ea86ca9e2f6/6cd00c1a-14cd-4705-8fa1-76b1c50e2463"
-					(reference "R31")
+					(reference "R66")
 					(unit 1)
 				)
@@
 		(dnp no)
 		(fields_autoplaced yes)
-		(property "Reference" "R56"
+		(property "Reference" "R69"
 			(at 179.07 59.69 90)
 			(effects
@@
 			(project "RC-Car-Project"
 				(path "/ba870fd1-751d-4755-8e1a-1ea86ca9e2f6/6cd00c1a-14cd-4705-8fa1-76b1c50e2463"
-					(reference "R56")
+					(reference "R69")
 					(unit 1)
 				)
@@
 		(dnp no)
 		(fields_autoplaced yes)
-		(property "Reference" "#PWR0128"
+		(property "Reference" "#PWR0153"
 			(at 185.42 113.03 0)
 			(effects
@@
 			(project "RC-Car-Project"
 				(path "/ba870fd1-751d-4755-8e1a-1ea86ca9e2f6/6cd00c1a-14cd-4705-8fa1-76b1c50e2463"
-					(reference "#PWR0128")
+					(reference "#PWR0153")
 					(unit 1)
 				)
@@
 		(dnp no)
 		(fields_autoplaced yes)
-		(property "Reference" "#PWR0129"
+		(property "Reference" "#PWR0154"
 			(at 195.58 81.28 0)
 			(effects
@@
 			(project "RC-Car-Project"
 				(path "/ba870fd1-751d-4755-8e1a-1ea86ca9e2f6/6cd00c1a-14cd-4705-8fa1-76b1c50e2463"
-					(reference "#PWR0129")
+					(reference "#PWR0154")
 					(unit 1)
 				)
@@
 		(dnp no)
 		(fields_autoplaced yes)
-		(property "Reference" "Q6"
+		(property "Reference" "Q7"
 			(at 140.97 97.7899 0)
 			(effects
@@
 			(project "RC-Car-Project"
 				(path "/ba870fd1-751d-4755-8e1a-1ea86ca9e2f6/6cd00c1a-14cd-4705-8fa1-76b1c50e2463"
-					(reference "Q6")
+					(reference "Q7")
 					(unit 1)
 				)
@@
 		(dnp no)
 		(fields_autoplaced yes)
-		(property "Reference" "#PWR0127"
+		(property "Reference" "#PWR0152"
 			(at 185.42 80.01 0)
 			(effects
@@
 			(project "RC-Car-Project"
 				(path "/ba870fd1-751d-4755-8e1a-1ea86ca9e2f6/6cd00c1a-14cd-4705-8fa1-76b1c50e2463"
-					(reference "#PWR0127")
+					(reference "#PWR0152")
 					(unit 1)
 				)
@@
 		(dnp no)
 		(fields_autoplaced yes)
-		(property "Reference" "#PWR0126"
+		(property "Reference" "#PWR0151"
 			(at 137.16 114.3 0)
 			(effects
@@
 			(project "RC-Car-Project"
 				(path "/ba870fd1-751d-4755-8e1a-1ea86ca9e2f6/6cd00c1a-14cd-4705-8fa1-76b1c50e2463"
-					(reference "#PWR0126")
+					(reference "#PWR0151")
 					(unit 1)
 				)
@@
 		(dnp no)
 		(fields_autoplaced yes)
-		(property "Reference" "R32"
+		(property "Reference" "R67"
 			(at 129.54 68.5799 0)
 			(effects
@@
 			(project "RC-Car-Project"
 				(path "/ba870fd1-751d-4755-8e1a-1ea86ca9e2f6/6cd00c1a-14cd-4705-8fa1-76b1c50e2463"
-					(reference "R32")
+					(reference "R67")
 					(unit 1)
 				)
@@
 		(dnp no)
 		(fields_autoplaced yes)
-		(property "Reference" "R58"
+		(property "Reference" "R71"
 			(at 187.96 68.5799 0)
 			(effects
@@
 			(project "RC-Car-Project"
 				(path "/ba870fd1-751d-4755-8e1a-1ea86ca9e2f6/6cd00c1a-14cd-4705-8fa1-76b1c50e2463"
-					(reference "R58")
+					(reference "R71")
 					(unit 1)
 				)
@@
 		(dnp no)
 		(fields_autoplaced yes)
-		(property "Reference" "#PWR0130"
+		(property "Reference" "#PWR0155"
 			(at 195.58 114.3 0)
 			(effects
@@
 			(project "RC-Car-Project"
 				(path "/ba870fd1-751d-4755-8e1a-1ea86ca9e2f6/6cd00c1a-14cd-4705-8fa1-76b1c50e2463"
-					(reference "#PWR0130")
+					(reference "#PWR0155")
 					(unit 1)
 				)
@@
 		(dnp no)
 		(fields_autoplaced yes)
-		(property "Reference" "Q5"
+		(property "Reference" "Q6"
 			(at 140.97 64.7699 0)
 			(effects
@@
 			(project ""
 				(path "/ba870fd1-751d-4755-8e1a-1ea86ca9e2f6/6cd00c1a-14cd-4705-8fa1-76b1c50e2463"
-					(reference "Q5")
+					(reference "Q6")
 					(unit 1)
 				)
@@
 		(dnp no)
 		(fields_autoplaced yes)
-		(property "Reference" "#PWR0124"
+		(property "Reference" "#PWR0149"
 			(at 127 113.03 0)
 			(effects
@@
 			(project "RC-Car-Project"
 				(path "/ba870fd1-751d-4755-8e1a-1ea86ca9e2f6/6cd00c1a-14cd-4705-8fa1-76b1c50e2463"
-					(reference "#PWR0124")
+					(reference "#PWR0149")
 					(unit 1)
 				)
@@
 		(dnp no)
 		(fields_autoplaced yes)
-		(property "Reference" "R59"
+		(property "Reference" "R72"
 			(at 187.96 101.5999 0)
 			(effects
@@
 			(project "RC-Car-Project"
 				(path "/ba870fd1-751d-4755-8e1a-1ea86ca9e2f6/6cd00c1a-14cd-4705-8fa1-76b1c50e2463"
-					(reference "R59")
-					(unit 1)
-				)
+					(reference "R72")
+					(unit 1)
+				)

Commit message: Most components speced
Parts:
- Q6, Q7, Q8, Q9: MANUF_PN (none) -> PMF250XNEX
Changed lines of the file:
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@@
 			)
 		)
-		(property "MANUF_PN" ""
+		(property "MANUF_PN" "PMF250XNEX"
 			(at 134.62 99.06 0)
 			(effects
@@
 			)
 		)
-		(property "MANUF_PN" ""
+		(property "MANUF_PN" "PMF250XNEX"
 			(at 193.04 99.06 0)
 			(effects
@@
 			)
 		)
-		(property "MANUF_PN" ""
+		(property "MANUF_PN" "PMF250XNEX"
 			(at 134.62 66.04 0)
 			(effects
@@
 			)
 		)
-		(property "MANUF_PN" ""
+		(property "MANUF_PN" "PMF250XNEX"
 			(at 193.04 66.04 0)
 			(effects
