File: RC-Car-Project/MotorDriver.kicad_sch (KiCad schematic)
At the start: 28 parts, among them Q1 BTN8982TA, Q2 BTN8982TA, Q3 BTN8982TA, Q4 BTN8982TA, U9 SN74HC244PWR

Commit message: Fixed (AGAIN AGAIN)
Parts:
- renumbered C44 to C41, C46 to C42, C45 to C43, C47 to C44, C48 to C45, Q1 to Q3, Q3 to Q4, Q4 to Q5, R62 to R47, R72 to R48, R22 to R49, R24 to R50, R23 to R51, R25 to R52, R64 to R53, R69 to R54, R27 to R55, R65 to R56, R68 to R57, R26 to R58, R66 to R59, R70 to R60, R28 to R61, R67 to R62, R71 to R63, R29 to R64, U9 to U8

Commit message: Most components speced
Parts:
- Q2, Q3, Q4, Q5: MANUF_PN (none) -> BTN8982TAAUMA1
- U8: MANUF_PN (none) -> SN74HC244PWR
Changed lines of the file:
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@@
 			)
 		)
-		(property "MANUF_PN" ""
+		(property "MANUF_PN" "BTN8982TAAUMA1"
 			(at 213.36 29.21 0)
 			(effects
@@
 			)
 		)
-		(property "MANUF_PN" ""
+		(property "MANUF_PN" "BTN8982TAAUMA1"
 			(at 213.36 104.14 0)
 			(effects
@@
 			)
 		)
-		(property "MANUF_PN" ""
+		(property "MANUF_PN" "BTN8982TAAUMA1"
 			(at 213.36 67.31 0)
 			(effects
@@
 			)
 		)
-		(property "MANUF_PN" ""
+		(property "MANUF_PN" "BTN8982TAAUMA1"
 			(at 213.36 135.89 0)
 			(effects
@@
 			)
 		)
-		(property "MANUF_PN" ""
+		(property "MANUF_PN" "SN74HC244PWR"
 			(at 69.85 71.12 0)
 			(effects
