File: RC-Car-Project/RC-Car-Project.kicad_sch (KiCad schematic)
At the start: 18 parts

Commit message: Fixed it (AGAIN!)
Parts:
- removed D1: LED, LED_SMD:LED_0603_1608Metric, symbol Device:LED
- removed R1, R60: 1.5kohm, Resistor_SMD:R_0603_1608Metric, symbol Device:R
- removed R2: 220ohm, Resistor_SMD:R_0603_1608Metric, symbol Device:R
- added D1 (x2): LED, LED_SMD:LED_0603_1608Metric, symbol Device:LED
- added R60 (x2): 1.5kohm, Resistor_SMD:R_0603_1608Metric, symbol Device:R
- added TP6: TestPoint, Connector_PinHeader_2.54mm:PinHeader_1x02_P2.54mm_Vertical, symbol Connector:TestPoint
Connections:
- net +12V: now also R60.1, R60.1
- net +3V3: now also TP6.1
- net GNDA: now also D1.1 (K), D1.1 (K)
- net at D11.2 (A): now also R60.2, R60.2
- net at R1.2: now also D1.2 (A), D1.2 (A)

Commit message: Fixed (AGAIN AGAIN)
Parts:
- removed D1: LED, LED_SMD:LED_0603_1608Metric, symbol Device:LED
- removed R60: 1.5kohm, Resistor_SMD:R_0603_1608Metric, symbol Device:R
- renumbered C56 to C1, C57 to C2, D11 to D1, D10 to D2, D1 to D3, D2 to D4, R60 to R1, R55 to R2, R1 to R3, R2 to R4, TP8 to TP1

Commit message: Most components speced
Parts:
- D1, D2, D3, D4: MANUF_PN (none) -> LTST-C190GKT
Changed lines of the file:
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@@
 			)
 		)
-		(property "MANUF_PN" ""
+		(property "MANUF_PN" "LTST-C190GKT"
 			(at 124.46 43.18 0)
 			(effects
@@
 			)
 		)
-		(property "MANUF_PN" ""
+		(property "MANUF_PN" "LTST-C190GKT"
 			(at 148.59 43.18 0)
 			(effects
@@
 			)
 		)
-		(property "MANUF_PN" ""
+		(property "MANUF_PN" "LTST-C190GKT"
 			(at 160.02 43.18 0)
 			(effects
@@
 			)
 		)
-		(property "MANUF_PN" ""
+		(property "MANUF_PN" "LTST-C190GKT"
 			(at 137.16 43.18 0)
 			(effects

Commit message: Add NA
Parts:
- TP1, TP2, TP3, TP4, TP5, TP6, TP7: MANUF_PN (none) -> N/A
Changed lines of the file:
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@@
+			)
+		)
+		(property "MANUF_PN" "N/A"
+			(at 208.28 31.75 0)
+			(effects
+				(font
+					(size 1.27 1.27)
+				)
+				(hide yes)
 			)
 		)
@@
 			)
 		)
+		(property "MANUF_PN" "N/A"
+			(at 186.69 31.75 0)
+			(effects
+				(font
+					(size 1.27 1.27)
+				)
+				(hide yes)
+			)
+		)
 		(pin "1"
 		)
@@
 			)
 		)
+		(property "MANUF_PN" "N/A"
+			(at 196.85 31.75 0)
+			(effects
+				(font
+					(size 1.27 1.27)
+				)
+				(hide yes)
+			)
+		)
 		(pin "1"
 		)
@@
 			)
 		)
+		(property "MANUF_PN" "N/A"
+			(at 176.53 31.75 0)
+			(effects
+				(font
+					(size 1.27 1.27)
+				)
+				(hide yes)
+			)
+		)
 		(pin "1"
 		)
@@
 			)
 		)
+		(property "MANUF_PN" "N/A"
+			(at 208.28 45.72 0)
+			(effects
+				(font
+					(size 1.27 1.27)
+				)
+				(hide yes)
+			)
+		)
 		(pin "1"
 		)
@@
 			)
 		)
+		(property "MANUF_PN" "N/A"
+			(at 186.69 45.72 0)
+			(effects
+				(font
+					(size 1.27 1.27)
+				)
+				(hide yes)
+			)
+		)
 		(pin "1"
 		)
@@
 			(at 196.85 45.72 0)
 			(effects
+				(font
+					(size 1.27 1.27)
+				)
+				(hide yes)
+			)
+		)
+		(property "MANUF_PN" "N/A"
+			(at 196.85 45.72 0)
+			(effects

Commit message: calc led resistors
Parts:
- R1: value 1.5kohm -> 2kohm; MANUF_PN RC0603JR-071K5L -> ERJ-2RKF2001X
- R2: value 220ohm -> 600ohm; MANUF_PN RMCF0603FT220R -> ERJ-3EKF5600V
- R3: value 1.5kohm -> 5kohm; MANUF_PN RC0603JR-071K5L -> RT0603BRE075KL
Changed lines of the file:
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@@
 			)
 		)
-		(property "Value" "1.5kohm"
+		(property "Value" "2kohm"
 			(at 126.238 36.322 0)
 			(effects
@@
 			)
 		)
-		(property "MANUF_PN" "RC0603JR-071K5L"
+		(property "MANUF_PN" "ERJ-2RKF2001X"
 			(at 161.29 35.56 0)
 			(effects
@@
 			)
 		)
-		(property "Value" "1.5kohm"
+		(property "Value" "5kohm"
 			(at 151.13 36.8299 0)
 			(effects
@@
 			)
 		)
-		(property "MANUF_PN" "RC0603JR-071K5L"
+		(property "MANUF_PN" "RT0603BRE075KL"
 			(at 148.59 35.56 0)
 			(effects
@@
 			)
 		)
-		(property "Value" "220ohm"
+		(property "Value" "600ohm"
 			(at 139.7 36.8299 0)
 			(effects
@@
 			)
 		)
-		(property "MANUF_PN" "RMCF0603FT220R"
+		(property "MANUF_PN" "ERJ-3EKF5600V"
 			(at 173.99 35.56 0)
 			(effects

Commit message: Finished BOM Drafts
Parts:
- R1: MANUF_PN ERJ-2RKF2001X -> ERA-3AEB202V
Changed lines of the file:
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@@
 			)
 		)
-		(property "MANUF_PN" "ERJ-2RKF2001X"
+		(property "MANUF_PN" "ERA-3AEB202V"
 			(at 161.29 35.56 0)
 			(effects

Commit message: Pushed pre-production things
Parts:
- added C46: C_Polarized, Inductor_THT:L_Radial_D12.0mm_P5.00mm_Neosid_SD12k_style2, symbol Device:C_Polarized
- C1, C2: MANUF_PN UHE2A101MPD1TD -> EEU-FS2A151LB
Connections:
- net GND_BATT: now also C46.2
- net VDD_BATT: now also C46.1
Changed lines of the file:
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@@
 	)
 	(junction
+		(at 104.14 43.18)
+		(diameter 0)
+		(color 0 0 0 0)
+	)
+	(junction
+		(at 104.14 35.56)
+		(diameter 0)
+		(color 0 0 0 0)
+	)
+	(junction
 		(at 97.79 43.18)
 		(diameter 0)
@@
 		)
 	)
+	(wire
+		(pts
+			(xy 104.14 35.56) (xy 110.49 35.56)
+		)
+		(stroke
+			(width 0)
+			(type default)
+		)
+	)
 	(bus
 		(pts
@@
 	(wire
 		(pts
+			(xy 104.14 43.18) (xy 110.49 43.18)
+		)
+		(stroke
+			(width 0)
+			(type default)
+		)
+	)
+	(wire
+		(pts
 			(xy 44.45 58.42) (xy 209.55 58.42)
 		)
@@
 			)
 		)
-		(property "MANUF_PN" "UHE2A101MPD1TD"
+		(property "MANUF_PN" "EEU-FS2A151LB"
 			(at 134.62 38.1 0)
 			(effects
@@
 	)
 	(symbol
+		(lib_id "Device:C_Polarized")
+		(at 110.49 39.37 0)
+		(unit 1)
+		(exclude_from_sim no)
+		(in_bom yes)
+		(on_board yes)
+		(dnp no)
+		(property "Reference" "C46"
+			(at 111.76 36.83 0)
+			(effects
+				(font
+					(size 1.27 1.27)
+				)
+				(justify left)
+			)
+		)
+		(property "Value" "C_Polarized"
+			(at 110.998 42.418 0)
+			(effects
+				(font
+					(size 1.27 1.27)
+				)
+				(justify left)
+			)
+		)
+		(property "Footprint" "Inductor_THT:L_Radial_D12.0mm_P5.00mm_Neosid_SD12k_style2"
+			(at 111.4552 43.18 0)
+			(effects
+				(font
+					(size 1.27 1.27)
+				)
+				(hide yes)
+			)
+		)
+		(property "Datasheet" "~"
+			(at 110.49 39.37 0)
+			(effects
+				(font
+					(size 1.27 1.27)
+				)
+				(hide yes)
+			)
+		)
+		(property "Description" "Polarized capacitor"
+			(at 110.49 39.37 0)
+			(effects
+				(font
+					(size 1.27 1.27)
+				)
+				(hide yes)
+			)
+		)
+		(property "MANUF_PN" "100ZLJ330M12.5X35"
+			(at 147.32 38.1 0)
+			(effects
+				(font
+					(size 1.27 1.27)
+				)
+				(hide yes)
+			)
+		)
+		(pin "1"
+		)
+		(pin "2"
+		)
+		(instances
+			(project "RC-Car-Project"
+				(path "/ba870fd1-751d-4755-8e1a-1ea86ca9e2f6"
+					(reference "C46")
+					(unit 1)
+				)
+			)
+		)
+	)
+	(symbol
 		(lib_id "power:+3V3")
 		(at 176.53 31.75 0)
@@
 		(on_board yes)
 		(dnp no)
-		(fields_autoplaced yes)
 		(property "Reference" "C2"
-			(at 107.95 37.2109 0)
+			(at 104.902 37.084 0)
 			(effects
 				(font
@@
 		)
 		(property "Value" "C_Polarized"
-			(at 107.95 39.7509 0)
+			(at 99.822 44.704 0)
 			(effects
 				(font
@@
 			)
 		)
-		(property "MANUF_PN" "UHE2A101MPD1TD"
+		(property "MANUF_PN" "EEU-FS2A151LB"
 			(at 140.97 38.1 0)
 			(effects
