File: RC-Car-Project/Connectors_sch.kicad_sch (KiCad schematic)
At the start: 21 parts, among them J1 Conn_01x02_Pin, J10 ANT_IF, J11 Conn_01x02, J12 Conn_01x02, J13 RF_IF, J14 Conn_01x02, J15 USB4120-03-C_REVA, J16 Conn_01x02, J2 Conn_01x02_Pin, J3 Conn_01x02_Pin, J4 Conn_01x02_Pin, J5 MCU_IF, J6 Conn_01x02, J7 Conn_01x02, J8 Conn_01x02, J9 Conn_02x09_Odd_Even, U4 USBLC6-2SC6

Commit message: Fixed (AGAIN AGAIN)
Parts:
- renumbered J11 to J10, J9 to J11, J5 to J12, J15 to J14, J10 to J15, J12 to J16, J6 to J5, J7 to J6, J14 to J7, J16 to J8, J8 to J9, R3 to R5, R4 to R6, R53 to R7, R54 to R8, U4 to U1

Commit message: Most components speced
Parts:
- J14: MANUF_PN (none) -> USB4120-03-C
Changed lines of the file:
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@@
 			)
 		)
-		(property "MANUF_PN" ""
+		(property "MANUF_PN" "USB4120-03-C"
 			(at 173.99 50.8 0)
 			(effects

Commit message: Add NA
Parts:
- J1, J2, J3, J4: MANUF_PN (none) -> N/A
Changed lines of the file:
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@@
 			)
 		)
-		(property "MANUF_PN" ""
+		(property "MANUF_PN" "N/A"
 			(at 78.74 119.38 0)
 			(effects
@@
 			)
 		)
-		(property "MANUF_PN" ""
+		(property "MANUF_PN" "N/A"
 			(at 78.74 128.27 0)
 			(effects
@@
 			)
 		)
-		(property "MANUF_PN" ""
+		(property "MANUF_PN" "N/A"
 			(at 78.74 104.14 0)
 			(effects
@@
 			)
 		)
-		(property "MANUF_PN" ""
+		(property "MANUF_PN" "N/A"
 			(at 78.74 95.25 0)
 			(effects

Commit message: Finished Rev1
Parts:
- J11: MANUF_PN PPPC092LFBN-RC -> PPPC092LJBN-RC
Changed lines of the file:
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@@
 			)
 		)
-		(property "MANUF_PN" "PPPC092LFBN-RC"
+		(property "MANUF_PN" "PPPC092LJBN-RC"
 			(at 85.09 44.45 0)
 			(effects
