File: RC-Car-Controller/CurrentSense.kicad_sch (KiCad schematic)
At the start: 7 parts, among them U8 INA229AQDGSRQ1

Commit message: Fixed Controller PCB
Parts:
- C3, C4: footprint (none) -> Capacitor_SMD:C_0201_0603Metric
- R15: footprint WSL2726_VIS -> footprints:WSL2726_VIS
- R2, R3, R4: footprint (none) -> Resistor_SMD:R_0201_0603Metric
- U8: footprint VSSOP10_DGS_TEX -> footprints:VSSOP10_DGS_TEX
Changed lines of the file:
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@@
 			)
 		)
-		(property "Footprint" "WSL2726_VIS"
+		(property "Footprint" "footprints:WSL2726_VIS"
 			(at 195.58 80.01 0)
 			(effects
@@
 			)
 		)
-		(property "Footprint" ""
+		(property "Footprint" "Resistor_SMD:R_0201_0603Metric"
 			(at 186.69 93.218 90)
 			(effects
@@
 			)
 		)
-		(property "Footprint" ""
+		(property "Footprint" "Capacitor_SMD:C_0201_0603Metric"
 			(at 169.8752 90.17 0)
 			(effects
@@
 			)
 		)
-		(property "Footprint" "VSSOP10_DGS_TEX"
+		(property "Footprint" "footprints:VSSOP10_DGS_TEX"
 			(at 113.03 86.36 0)
 			(effects
@@
 			)
 		)
-		(property "Footprint" ""
+		(property "Footprint" "Resistor_SMD:R_0201_0603Metric"
 			(at 186.69 84.328 90)
 			(effects
@@
 			)
 		)
-		(property "Footprint" ""
+		(property "Footprint" "Resistor_SMD:R_0201_0603Metric"
 			(at 94.742 87.63 90)
 			(effects
@@
 			)
 		)
-		(property "Footprint" ""
+		(property "Footprint" "Capacitor_SMD:C_0201_0603Metric"
 			(at 157.1752 104.14 0)
 			(effects
