File: RC-Car-Controller/MotorDriver.kicad_sch (KiCad schematic)
At the start: 14 parts, among them Q1 BTN8982TA, Q2 BTN8982TA, Q5 BTN8982TA, Q6 BTN8982TA, U9 SN74HC244PWR

Commit message: Fixed Controller PCB
Parts:
- C13, C41, C42, C5, C6: footprint (none) -> Capacitor_SMD:C_0201_0603Metric
- R17, R18, R5, R6: footprint (none) -> Resistor_SMD:R_0201_0603Metric
- U9: footprint PW20 -> footprints:PW20
Connections:
- net MOTOR_1_L_EN: no longer U9.2 (1A1)
- net MOTOR_1_L_PWM: no longer U9.4 (1A2)
- net MOTOR_1_R_EN: no longer U9.6 (1A3)
- net MOTOR_1_R_PWM: no longer U9.8 (1A4)
- new net MOTOR_2_L_EN: U9.2 (1A1)
- new net MOTOR_2_L_PWM: U9.4 (1A2)
- new net MOTOR_2_R_EN: U9.6 (1A3)
- new net MOTOR_2_R_PWM: U9.8 (1A4)
Changed lines of the file:
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@@
 		)
 	)
-	(hierarchical_label "MOTOR_1_R_PWM"
+	(hierarchical_label "MOTOR_2_R_PWM"
 		(shape input)
 		(at 69.85 100.33 180)
@@
 		)
 	)
-	(hierarchical_label "MOTOR_1_L_PWM"
+	(hierarchical_label "MOTOR_2_L_PWM"
 		(shape input)
 		(at 69.85 90.17 180)
@@
 		)
 	)
-	(hierarchical_label "MOTOR_1_L_EN"
+	(hierarchical_label "MOTOR_2_L_EN"
 		(shape input)
 		(at 69.85 85.09 180)
@@
 		)
 	)
-	(hierarchical_label "MOTOR_1_R_EN"
+	(hierarchical_label "MOTOR_2_R_EN"
 		(shape input)
 		(at 69.85 95.25 180)
@@
 			)
 		)
-		(property "Footprint" ""
+		(property "Footprint" "Capacitor_SMD:C_0201_0603Metric"
 			(at 145.7452 80.01 0)
 			(effects
@@
 			)
 		)
-		(property "Footprint" ""
+		(property "Footprint" "Resistor_SMD:R_0201_0603Metric"
 			(at 200.152 144.78 90)
 			(effects
@@
 			)
 		)
-		(property "Footprint" ""
+		(property "Footprint" "Capacitor_SMD:C_0201_0603Metric"
 			(at 191.4652 48.26 0)
 			(effects
@@
 			)
 		)
-		(property "Footprint" ""
+		(property "Footprint" "Resistor_SMD:R_0201_0603Metric"
 			(at 200.152 44.45 90)
 			(effects
@@
 			)
 		)
-		(property "Footprint" ""
+		(property "Footprint" "Resistor_SMD:R_0201_0603Metric"
 			(at 200.152 76.2 90)
 			(effects
@@
 			)
 		)
-		(property "Footprint" "PW20"
+		(property "Footprint" "footprints:PW20"
 			(at 69.85 82.55 0)
 			(effects
@@
 			)
 		)
-		(property "Footprint" ""
+		(property "Footprint" "Resistor_SMD:R_0201_0603Metric"
 			(at 200.152 113.03 90)
 			(effects
@@
 			)
 		)
-		(property "Footprint" ""
+		(property "Footprint" "Capacitor_SMD:C_0201_0603Metric"
 			(at 191.4652 116.84 0)
 			(effects
@@
 			)
 		)
-		(property "Footprint" ""
+		(property "Footprint" "Capacitor_SMD:C_0201_0603Metric"
 			(at 191.4652 80.01 0)
 			(effects
@@
 			)
 		)
-		(property "Footprint" ""
+		(property "Footprint" "Capacitor_SMD:C_0201_0603Metric"
 			(at 191.4652 148.59 0)
 			(effects
