File: RC-Car-Controller/Power_sch.kicad_sch (KiCad schematic)
At the start: 30 parts, among them Q1 DMG2301L, U10 STC3100IST, U8 BQ25303JRTER, U9 AP63203WU

Commit message: Did power schtuff
Parts:
- removed C36: 100nF/16V, Capacitor_SMD:C_0603_1608Metric, symbol Device:C
- removed C37, C38: 22uF/16V, Capacitor_SMD:C_0603_1608Metric, symbol Device:C
- removed C39: 10uF/16V, Capacitor_SMD:C_0603_1608Metric, symbol Device:C
- removed U9: AP63203WU, Package_TO_SOT_SMD:TSOT-23-6, symbol Regulator_Switching:AP63203WU
- added C18: 3.3nF/10V, Capacitor_SMD:C_0603_1608Metric, symbol Device:C
- added C19: 0.1uF/10V, Capacitor_SMD:C_0603_1608Metric, symbol Device:C
- added C20: 10uF/10V, Capacitor_SMD:C_1210_3225Metric, symbol Device:C
- added C22: 22uF/10V, Capacitor_SMD:C_0805_2012Metric, symbol Device:C
- added R18: 100kohm, Resistor_SMD:R_0603_1608Metric, symbol Device:R
- added U1: TPS62132, Package_DFN_QFN:VQFN-16-1EP_3x3mm_P0.5mm_EP1.68x1.68mm_ThermalVias, symbol Regulator_Switching:TPS62132
- C14: value 2.2uF/16V -> 2.2uF/10V
- C15: value 47nF/16V -> 47nF/10V
- C16, C2: value 10uF/16V -> 10uF/10V
- L2: value 3.9uH -> 2.2uH
- R9: value 1.5kohm -> 1kohm
- U10: footprint MiniSO8_STM -> STC3100IST:MiniSO8_STM
Connections:
- net +3V3: now also C22.2, R18.2, U1.14 (VOS)
- net GNDA: now also C18.1, C19.1, C20.1, C22.1, U1.15 (GND), U1.16 (GND), U1.17 (GND), U1.5 (FB), U1.6 (GND), U1.7 (FSW), U1.8 (DEF)
- net VDD_LOAD: now also C19.2, C20.2, U1.10 (VIN), U1.11 (VIN), U1.12 (VIN), U1.13 (EN)
- net VDD_LOAD_PRE_SW: now also C2.2, U8.16 (PMID); no longer D5.1 (K)
- net VDD_USB: no longer Q1.1 (G)
- net at L2.1: now also U1.1 (SW), U1.2 (SW), U1.3 (SW)
- new net: R18.1, U1.4 (PG)
- new net: C18.2, U1.9 (SS/TR)
- new net: D5.1 (K), Q1.1 (G)
Other:
- note removed: "3V3 Regulator [TO BE REPLACED]"
- moved on the sheet: D5, Q1

Commit message: Did a bunch of stuff on the controller
Parts:
- removed R5, R6: 10kohm, Resistor_SMD:R_0603_1608Metric, symbol Device:R
- R14, R15: footprint Resistor_SMD:R_0603_1608Metric -> Capacitor_SMD:C_0603_1608Metric

Commit message: Finished Controller PCB Pre-Review
Parts:
- R15: renamed from R1; footprint Resistor_SMD:R_0603_1608Metric -> Resistor_SMD:R_0805_2012Metric
- R8: renamed from R9; value 1kohm -> 220ohm
- renumbered C17 to C10, C3 to C11, C14 to C3, C20 to C4, C19 to C5, C18 to C6, C15 to C7, C22 to C8, C16 to C9, L2 to L1, L1 to L2, R14 to R10, R18 to R11, R15 to R12, R22 to R13, R4 to R14, R21 to R6, R10 to R7, R13 to R9, U8 to U2, U1 to U3, U10 to U4
