File: RC-Car-Controller/Power_sch.kicad_sch (KiCad schematic)
At the start: 29 parts, among them Q1 DMG2301L, U2 BQ25303JRTER, U3 TPS62132, U4 STC3100IST

Commit message: Controller Design Review
Parts:
- R7: value 20kohm -> 13kohm
- R8: value 220ohm -> 1kohm
Changed lines of the file:
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@@
 	(wire
 		(pts
-			(xy 97.79 152.4) (xy 97.79 160.02)
-		)
-		(stroke
-			(width 0)
-			(type default)
-		)
-	)
-	(wire
-		(pts
 			(xy 60.96 149.86) (xy 66.04 149.86)
 		)
@@
 	(wire
 		(pts
+			(xy 97.79 160.02) (xy 97.79 152.4)
+		)
+		(stroke
+			(width 0)
+			(type default)
+		)
+	)
+	(wire
+		(pts
 			(xy 105.41 91.44) (xy 107.95 91.44)
 		)
@@
 			)
 		)
-		(property "Value" "20kohm"
+		(property "Value" "13kohm"
 			(at 59.69 75.946 90)
 			(effects
@@
 			)
 		)
-		(property "Value" "220ohm"
+		(property "Value" "1kohm"
 			(at 59.69 85.852 90)
 			(effects

Commit message: most resistors given PNs
most resistors given PNs. some remaining
Parts:
- R10, R12: MANUF_PN (none) -> RC0603FR-0710KL
- R11, R6: MANUF_PN (none) -> RMCF0603FT100K
- R13: MANUF_PN (none) -> RG1608N-204-W-T1
- R14, R8: MANUF_PN (none) -> RMCF0603FT1K00
- R15: MANUF_PN (none) -> ERJ-6CWDR020V
- R9: MANUF_PN (none) -> RMCF0603FT220R

Commit message: controller cpnts given MANUF_PNs
controller cpnts given MANUF_PNs. not all components, but all resistors are done
Parts:
- D5: MANUF_PN (none) -> SK36A-LTP
- Q1: MANUF_PN (none) -> DMG2301L-7
- R7: MANUF_PN (none) -> RC0603FR-0713KL
- U2: MANUF_PN (none) -> BQ25303JRTER
- U3: MANUF_PN (none) -> TPS62132RGTR
- U4: MANUF_PN (none) -> STC3100IST
Changed lines of the file:
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@@
 			)
 		)
-		(property "MANUF_PN" ""
+		(property "MANUF_PN" "BQ25303JRTER"
 			(at 85.09 71.12 0)
 			(effects
@@
 			)
 		)
-		(property "MANUF_PN" ""
+		(property "MANUF_PN" "TPS62132RGTR"
 			(at 87.63 147.32 0)
 			(effects
@@
 			)
 		)
-		(property "MANUF_PN" ""
+		(property "MANUF_PN" "STC3100IST"
 			(at 196.85 53.34 0)
 			(effects
@@
 			)
 		)
-		(property "MANUF_PN" ""
+		(property "MANUF_PN" "RC0603FR-0713KL"
 			(at 59.69 73.66 0)
 			(effects
@@
 			)
 		)
-		(property "MANUF_PN" ""
+		(property "MANUF_PN" "DMG2301L-7"
 			(at 137.16 40.64 0)
 			(effects
@@
 			)
 		)
-		(property "MANUF_PN" ""
+		(property "MANUF_PN" "SK36A-LTP"
 			(at 128.27 40.64 0)
 			(effects

Commit message: Filled out some Controller Caps
Parts:
- C1: value 2.2uF/16V -> 2.2uF/10V; MANUF_PN (none) -> C0603C225K4PACTU
- C10: value 220nF/16V -> 0.22F/10V
- C11: value 1uF/16V -> 1uF/10V; MANUF_PN (none) -> CL10B105KO8NNNC
- C3: MANUF_PN (none) -> C0603C225K4PACTU
- C5: MANUF_PN (none) -> C0603C104K5RAC7411
- C8: MANUF_PN (none) -> CL21A226MPQNNNE
Changed lines of the file:
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@@
 			)
 		)
-		(property "MANUF_PN" ""
+		(property "MANUF_PN" "C0603C225K4PACTU"
 			(at 59.69 68.58 0)
 			(effects
@@
 			)
 		)
-		(property "MANUF_PN" ""
+		(property "MANUF_PN" "C0603C104K5RAC7411"
 			(at 66.04 138.43 0)
 			(effects
@@
 			)
 		)
-		(property "Value" "220nF/16V"
+		(property "Value" "0.22F/10V"
 			(at 244.856 47.244 0)
 			(effects
@@
 			)
 		)
-		(property "Value" "2.2uF/16V"
+		(property "Value" "2.2uF/10V"
 			(at 38.862 57.912 0)
 			(effects
@@
 			)
 		)
-		(property "MANUF_PN" ""
+		(property "MANUF_PN" "C0603C225K4PACTU"
 			(at 52.07 57.15 0)
 			(effects
@@
 			)
 		)
-		(property "MANUF_PN" ""
+		(property "MANUF_PN" "CL21A226MPQNNNE"
 			(at 125.73 146.05 0)
 			(effects
@@
 			)
 		)
-		(property "Value" "1uF/16V"
+		(property "Value" "1uF/10V"
 			(at 267.716 65.024 0)
 			(effects
@@
 			)
 		)
-		(property "MANUF_PN" ""
+		(property "MANUF_PN" "CL10B105KO8NNNC"
 			(at 266.7 62.23 0)
 			(effects

Commit message: Added Schem PNs
Parts:
- C10: value 0.22F/10V -> 0.22uF/10V; MANUF_PN (none) -> CC0603KRX7R6BB224
- C2, C9: MANUF_PN (none) -> CL10A106KP8NNNC
- C4: MANUF_PN (none) -> LMK325B7106KN-T
- C6: MANUF_PN (none) -> 885012206011
- C7: MANUF_PN (none) -> 885012206018
- L1: MANUF_PN (none) -> 74438357022
- L2: MANUF_PN (none) -> 74438357010
Changed lines of the file:
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@@
 			)
 		)
-		(property "MANUF_PN" ""
+		(property "MANUF_PN" "LMK325B7106KN-T"
 			(at 60.96 138.43 0)
 			(effects
@@
 			)
 		)
-		(property "MANUF_PN" ""
+		(property "MANUF_PN" "CL10A106KP8NNNC"
 			(at 59.69 60.96 0)
 			(effects
@@
 			)
 		)
-		(property "MANUF_PN" ""
+		(property "MANUF_PN" "CL10A106KP8NNNC"
 			(at 127 57.15 0)
 			(effects
@@
 			)
 		)
-		(property "MANUF_PN" ""
+		(property "MANUF_PN" "74438357010"
 			(at 119.38 53.34 0)
 			(effects
@@
 			)
 		)
-		(property "Value" "0.22F/10V"
+		(property "Value" "0.22uF/10V"
 			(at 244.856 47.244 0)
 			(effects
@@
 			)
 		)
-		(property "MANUF_PN" ""
+		(property "MANUF_PN" "CC0603KRX7R6BB224"
 			(at 243.84 44.45 0)
 			(effects
@@
 			)
 		)
-		(property "MANUF_PN" ""
+		(property "MANUF_PN" "885012206018"
 			(at 111.76 57.15 0)
 			(effects
@@
 			)
 		)
-		(property "MANUF_PN" ""
+		(property "MANUF_PN" "885012206011"
 			(at 73.66 144.78 0)
 			(effects
@@
 			)
 		)
-		(property "MANUF_PN" ""
+		(property "MANUF_PN" "74438357022"
 			(at 101.6 142.24 0)
 			(effects

Commit message: Finished BOM Drafts
Parts:
- D4: MANUF_PN (none) -> LTST-C190GKT
- R8: value 1kohm -> 220ohm; MANUF_PN RMCF0603FT1K00 -> RMCF0603FT220R
Changed lines of the file:
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@@
 	)
 	(junction
+		(at 266.7 55.88)
+		(diameter 0)
+		(color 0 0 0 0)
+	)
+	(junction
 		(at 64.77 68.58)
 		(diameter 0)
@@
 	)
 	(junction
-		(at 266.7 55.88)
-		(diameter 0)
-		(color 0 0 0 0)
-	)
-	(junction
 		(at 76.2 149.86)
 		(diameter 0)
@@
 	(wire
 		(pts
-			(xy 243.84 55.88) (xy 266.7 55.88)
-		)
-		(stroke
-			(width 0)
-			(type default)
-		)
-	)
-	(wire
-		(pts
 			(xy 139.7 66.04) (xy 105.41 66.04)
 		)
@@
 	(wire
 		(pts
+			(xy 243.84 55.88) (xy 266.7 55.88)
+		)
+		(stroke
+			(width 0)
+			(type default)
+		)
+	)
+	(wire
+		(pts
 			(xy 69.85 149.86) (xy 76.2 149.86)
 		)
@@
 	(wire
 		(pts
-			(xy 266.7 55.88) (xy 266.7 48.26)
+			(xy 63.5 83.82) (xy 64.77 83.82)
 		)
 		(stroke
@@
 	(wire
 		(pts
-			(xy 63.5 83.82) (xy 64.77 83.82)
+			(xy 60.96 149.86) (xy 66.04 149.86)
 		)
 		(stroke
@@
 	(wire
 		(pts
-			(xy 60.96 149.86) (xy 66.04 149.86)
+			(xy 55.88 68.58) (xy 52.07 68.58)
 		)
 		(stroke
@@
 	(wire
 		(pts
-			(xy 55.88 68.58) (xy 52.07 68.58)
+			(xy 257.81 58.42) (xy 243.84 58.42)
 		)
 		(stroke
@@
 	(wire
 		(pts
-			(xy 257.81 58.42) (xy 243.84 58.42)
+			(xy 237.49 53.34) (xy 240.03 53.34)
 		)
 		(stroke
@@
 	(wire
 		(pts
-			(xy 237.49 53.34) (xy 240.03 53.34)
+			(xy 266.7 40.64) (xy 266.7 55.88)
 		)
 		(stroke
@@
 	(wire
 		(pts
-			(xy 176.53 55.88) (xy 177.8 55.88)
+			(xy 52.07 35.56) (xy 52.07 40.64)
 		)
 		(stroke
@@
 	(wire
 		(pts
-			(xy 52.07 40.64) (xy 52.07 35.56)
+			(xy 176.53 55.88) (xy 177.8 55.88)
 		)
 		(stroke
@@
 	(symbol
 		(lib_id "power:+3V3")
-		(at 266.7 48.26 0)
+		(at 266.7 40.64 0)
 		(unit 1)
 		(exclude_from_sim no)
@@
 		(dnp no)
 		(property "Reference" "#PWR055"
-			(at 266.7 52.07 0)
+			(at 266.7 44.45 0)
 			(effects
 				(font
@@
 		)
 		(property "Value" "VDD_BATT"
-			(at 262.128 44.196 0)
+			(at 262.128 36.576 0)
 			(effects
 				(font
@@
 		)
 		(property "Footprint" ""
-			(at 266.7 48.26 0)
+			(at 266.7 40.64 0)
 			(effects
 				(font
@@
 		)
 		(property "Datasheet" ""
-			(at 266.7 48.26 0)
+			(at 266.7 40.64 0)
 			(effects
 				(font
@@
 		)
 		(property "Description" "Power symbol creates a global label with name \"+3V3\""
-			(at 266.7 48.26 0)
+			(at 266.7 40.64 0)
 			(effects
 				(font
@@
 			)
 		)
-		(property "MANUF_PN" ""
+		(property "MANUF_PN" "LTST-C190GKT"
 			(at 43.18 83.82 0)
 			(effects
@@
 			)
 		)
-		(property "Value" "1kohm"
+		(property "Value" "220ohm"
 			(at 59.69 85.852 90)
 			(effects
@@
 			)
 		)
-		(property "MANUF_PN" "RMCF0603FT1K00"
+		(property "MANUF_PN" "RMCF0603FT220R"
 			(at 59.69 83.82 0)
 			(effects

Commit message: Finished Rev1
Parts:
- D5: value SK36A-LTP -> SK54A-LTP; MANUF_PN SK36A-LTP -> SK54A-LTP
Changed lines of the file:
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@@
 			)
 		)
-		(property "Value" "SK36A-LTP"
+		(property "Value" "SK54A-LTP"
 			(at 124.46 37.592 0)
 			(effects
@@
 			)
 		)
-		(property "MANUF_PN" "SK36A-LTP"
+		(property "MANUF_PN" "SK54A-LTP"
 			(at 128.27 40.64 0)
 			(effects
