File: RC-Car-Controller/RC-Car-Controller.kicad_pcb (KiCad board)
At the start: 2 copper layers, 69 parts, among them J3 Conn_01x08_Pin, J4 Conn_01x02, J5 MCU_IF, J6 ANT_IF, Q1 PMOS, SW1 SW_Push, SW2 1825027-8, SW4 1825027-8, U1 AT86RF215-ZU, U2 A6986F3V3TR, U3 ADC082S021CIMM/NOPB, U4 STM32H743VGTx, U5 RFX2401C, U6 2450FB15A050E, Y1 Crystal

Commit message: Added a switch
Parts:
- removed C18, C19, C22: 10uF/50V, Capacitor_SMD:C_0603_1608Metric
- removed C20, C23: 1uF/50V, Capacitor_SMD:C_0603_1608Metric
- removed C34: 1uF/16V, Capacitor_SMD:C_0603_1608Metric
- removed J4: Conn_01x02, Connector_JST:JST_XH_B2B-XH-AM_1x02_P2.50mm_Vertical
- removed U3: ADC082S021CIMM/NOPB, footprints:MUA08A
- added C36: 100nF/16V, Capacitor_SMD:C_0603_1608Metric, F.Cu at (49.0, 112.4)
- added C37: 22uF/16V, Capacitor_SMD:C_0603_1608Metric, F.Cu at (49.0, 114.9)
- added C38: 22uF/16V, Capacitor_SMD:C_0603_1608Metric, F.Cu at (49.0, 117.4)
- added C39: 10uF/16V, Capacitor_SMD:C_0603_1608Metric, F.Cu at (49.0, 119.9)
- added D4: LED, LED_SMD:LED_0603_1608Metric, F.Cu at (55.2, 129.6)
- added D5: SK36A-LTP, Diode_SMD:D_SMA, F.Cu at (57.3, 126.0)
- added J1: Conn_01x02, Connector_JST:JST_XH_B2B-XH-AM_1x02_P2.50mm_Vertical, F.Cu at (57.8, 136.2)
- added J7: 2171790001, USB-C 2171790001:2171790001_MOL, F.Cu at (40.8, 147.0)
- added L2: 3.9uH, Inductor_SMD:L_Wuerth_MAPI-4030, F.Cu at (50.6, 126.4)
- added R21: 100kohm, Resistor_SMD:R_0603_1608Metric, F.Cu at (57.0, 114.9)
- added R22: 200kohm 0.1%, Resistor_SMD:R_0603_1608Metric, F.Cu at (57.0, 117.4)
- added R23: 5.11kohm, Resistor_SMD:R_0603_1608Metric, F.Cu at (37.2, 152.5)
- added R24: 5.11kohm, Resistor_SMD:R_0603_1608Metric, F.Cu at (37.2, 155.0)
- added R4: 1kohm, Resistor_SMD:R_0603_1608Metric, F.Cu at (53.0, 109.9)
- added R5: 10kohm, Resistor_SMD:R_0603_1608Metric, F.Cu at (53.0, 112.4)
- added S1: R1966ABLKBLKGR, R1966ABLKBLKGR:SW_R1966ABLKBLKGR, F.Cu at (188.2, 139.0)
- added U8: BQ25303JRTER, BQ25303JRTER:RTE0016C, F.Cu at (61.4, 120.2)
- added U9: AP63203WU, Package_TO_SOT_SMD:TSOT-23-6, F.Cu at (61.6, 111.0)
- C1: value 470nF/25V -> 2.2uF/16V
- C14: value 68nF/25V -> 2.2uF/16V
- C15: value 220pF/25V -> 47nF/16V
- C16: value 10nF/25V -> 10uF/16V
- C17: value 220pF/16V -> 220nF/16V
- C2: value 220pF/25V -> 10uF/16V
- C3: value 0.1uF/10V -> 1uF/16V; footprint Capacitor_SMD:C_0201_0603Metric -> Capacitor_SMD:C_0603_1608Metric
- L1: value 8.2uH -> 1uH
- Q1: value PMOS -> DMG2301L; footprint Package_TO_SOT_SMD:TO-263-2 -> Package_TO_SOT_SMD:SOT-23
- R1: value 68Kohm -> 20mohm 1%; footprint Resistor_SMD:R_0201_0603Metric -> Resistor_SMD:R_0603_1608Metric
- R10: value 75kohm -> 20kohm
- R13: value 1Mohm -> 220ohm
- R14: value 280kohm -> 10kohm
- R6: value 100Kohm -> 10kohm; footprint Resistor_SMD:R_0201_0603Metric -> Resistor_SMD:R_0603_1608Metric
- R9: value 1.8kohm -> 1.5kohm
- U2: value A6986F3V3TR -> USBLC6-2SC6; footprint footprints:HTSSOP16_4P5X5P1X0P65P_STM -> Package_TO_SOT_SMD:SOT-23-6
- moved L1 134.0 mm to (45.5, 126.4)
- moved C1 122.5 mm to (45.0, 109.9)
- moved C2 122.5 mm to (45.0, 112.4)
- moved C14 122.3 mm to (45.0, 117.4)
- moved C15 122.3 mm to (45.0, 119.9)
- moved C16 122.3 mm to (45.0, 122.5)
- moved R10 122.0 mm to (53.0, 119.9)
- moved R13 122.0 mm to (53.0, 122.5)
- moved R9 122.0 mm to (53.0, 117.4)
- moved U2 121.9 mm to (60.9, 143.1)
- moved C17 120.5 mm to (49.0, 109.9)
- moved R14 119.5 mm to (57.0, 109.9)
- moved R15 119.5 mm to (57.0, 112.4)
- moved Q1 114.1 mm to (61.5, 115.7)
- moved C3 77.7 mm to (45.0, 114.9)
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Connections:
- C1 pad 1: Net-(U2-MLF) -> VDD_USB
- C14 pad 1: Net-(U2-SS/*INH) -> GNDA
- C14 pad 2: GNDA -> /Power/REGN
- C15 pad 1: GNDA -> Net-(C15-Pad1)
- C15 pad 2: Net-(U2-COMP) -> Net-(U8-BTST)
- C16 pad 1: Net-(U2-DELAY) -> VDD_BATT
- C17 pad 1: +3V3 -> GNDA
- C17 pad 2: Net-(U2-VOUT) -> Net-(U10-VIN)
- C2 pad 2: Net-(C2-Pad2) -> Net-(U8-PMID)
- C3 pad 1: +3V3 -> VDD_BATT
- L1 pad 1: Net-(L1-Pad1) -> Net-(C15-Pad1)
- L1 pad 2: +3V3 -> VDD_BATT
- Q1 pad 1: VDD_BATT -> VDD_USB
- Q1 pad 2: /Connectors/PWR_SW -> VDD_LOAD_PRE_SW
- Q1 pad 3: VDD_BATT_PRE_SW -> VDD_BATT
- R1 pad 2: Net-(U3-IN1) -> GND_BATT
- R10 pad 1: Net-(C2-Pad2) -> GNDA
- R10 pad 2: Net-(U2-COMP) -> Net-(U8-ICHG)
- R12 pad 1: Net-(U4-BOOT0) -> unconnected-(R12-Pad1)
- R13 pad 1: Net-(U2-RST) -> GNDA
- R13 pad 2: +3V3 -> Net-(U8-VSET)
- R14 pad 1: Net-(U2-VOUT) -> Net-(U8-TS)
- R14 pad 2: +3V3 -> GNDA
- R15 pad 1: GNDA -> /Power/REGN
- R15 pad 2: Net-(U2-VOUT) -> Net-(U8-TS)
- R6 pad 1: Net-(U3-IN1) -> /Power/GAS_SDA
- R6 pad 2: VDD_REF -> +3V3
- R7 pad 1: VDD_BATT -> VDD_LOAD
- R9 pad 1: GNDA -> Net-(D4-K)
- R9 pad 2: Net-(U2-FSW) -> Net-(U8-STAT)
- U2 pad 1: Net-(U2-RST) -> Net-(J7-DP1)
- U2 pad 2: Net-(U2-MLF) -> GNDA
- U2 pad 3: Net-(U2-SS/*INH) -> Net-(J7-DN1)
- U2 pad 4: unconnected-(U2-SYNCH/ISKIP-Pad4) -> /Connectors/CON_USB_D-
- U2 pad 5: Net-(U2-FSW) -> VDD_USB
- U2 pad 6: Net-(U2-MLF) -> /Connectors/CON_USB_D+
- U4 pad 36: /ADC/MOSI -> /MCU/SPI3_MOSI
- U4 pad 70: unconnected-(U4-PA11-Pad70) -> /Connectors/CON_USB_D-
- U4 pad 71: unconnected-(U4-PA12-Pad71) -> /Connectors/CON_USB_D+
- U4 pad 78: /ADC/SCLK -> /MCU/SPI3_SCLK
- U4 pad 79: /ADC/MISO -> /MCU/SPI3_MISO
- U4 pad 80: /ADC/ADC_CS -> /MCU/SPI3_CS_ADC
- U4 pad 94: Net-(U4-BOOT0) -> unconnected-(U4-BOOT0-Pad94)
Other:
- board outline added: 8.6 x 5 mm

Commit message: Did power schtuff
Parts:
- removed C24, C25, C26, C27, C28, C29, C30, C31, C32, C33: 0.1uF/10V, Capacitor_SMD:C_0201_0603Metric
- removed C36: 100nF/16V, Capacitor_SMD:C_0603_1608Metric
- removed C37, C38: 22uF/16V, Capacitor_SMD:C_0603_1608Metric
- removed C39: 10uF/16V, Capacitor_SMD:C_0603_1608Metric
- removed U5: RFX2401C, footprints:RFX2401C_SKY
- removed U6: 2450FB15A050E, footprints:2450FB15A050E_JOT
- removed U9: AP63203WU, Package_TO_SOT_SMD:TSOT-23-6
- added C18: 3.3nF/10V, Capacitor_SMD:C_0603_1608Metric, F.Cu at (118.1, 87.0)
- added C19: 0.1uF/10V, Capacitor_SMD:C_0603_1608Metric, F.Cu at (117.3, 84.6)
- added C20: 10uF/10V, Capacitor_SMD:C_1210_3225Metric, F.Cu at (113.3, 83.8)
- added C22: 22uF/10V, Capacitor_SMD:C_0805_2012Metric, F.Cu at (111.9, 90.2)
- added R18: 100kohm, Resistor_SMD:R_0603_1608Metric, F.Cu at (118.1, 90.0)
- added U10: STC3100IST, STC3100IST:MiniSO8_STM, F.Cu at (106.1, 91.2)
- C14: value 2.2uF/16V -> 2.2uF/10V
- C15: value 47nF/16V -> 47nF/10V
- C16, C2: value 10uF/16V -> 10uF/10V
- L2: value 3.9uH -> 2.2uH
- R9: value 1.5kohm -> 1kohm
- U1: value AT86RF215-ZU -> TPS62132; footprint footprints:QFN48_PQ_MCH -> Package_DFN_QFN:VQFN-16-1EP_3x3mm_P0.5mm_EP1.68x1.68mm_ThermalVias
- moved R24 151.5 mm to (148.6, 52.3), turned to 90 degrees
- moved R23 145.5 mm to (142.7, 52.3), turned to 90 degrees
- moved J7 145.4 mm to (145.6, 46.3), turned to 180 degrees
- moved U2 123.4 mm to (145.6, 53.4), turned to -90 degrees
- moved S1 112.5 mm to (108.7, 59.4), turned to 180 degrees
- moved R6 85.7 mm to (129.5, 76.5)
- moved R5 85.3 mm to (129.5, 74.7)
- moved D4 82.8 mm to (115.8, 73.0), turned to -90 degrees
- moved D5 82.4 mm to (112.5, 64.9), turned to 90 degrees
- moved C14 81.1 mm to (114.6, 75.9), turned to 180 degrees
- moved C15 77.5 mm to (111.7, 80.5), turned to 90 degrees
- moved L1 77.3 mm to (108.8, 81.9), turned to 180 degrees
- moved C16 76.9 mm to (107.7, 77.8), turned to 90 degrees
- moved C1 76.8 mm to (114.6, 77.6)
- moved R10 75.7 mm to (112.5, 73.0), turned to -90 degrees
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Connections:
- C2 pad 2: Net-(U8-PMID) -> VDD_LOAD_PRE_SW
- D5 pad 1: VDD_LOAD_PRE_SW -> Net-(D5-K)
- J3 pad 3: /MCU/SPI2_MOSI -> /MCU/SPI4_MOSI
- J3 pad 4: /MCU/SPI2_SCLK -> /MCU/SPI4_SCLK
- J3 pad 5: /MCU/SPI2_CS_LCD -> /Outputs/LCD_CS
- L2 pad 1: Net-(U9-SW) -> Net-(L2-Pad1)
- Q1 pad 1: VDD_USB -> Net-(D5-K)
- R5 pad 1: /Power/GAS_SCL -> /MCU/I2C3_SCL
- R6 pad 1: /Power/GAS_SDA -> /MCU/I2C3_SDA
- U1 pad 1: /RF/RXEN -> Net-(L2-Pad1)
- U1 pad 10: GNDA -> VDD_LOAD
- U1 pad 11: unconnected-(U1-FEA09-Pad11) -> VDD_LOAD
- U1 pad 12: unconnected-(U1-FEB09-Pad12) -> VDD_LOAD
- U1 pad 13: /MCU/RF_NRST -> VDD_LOAD
- U1 pad 15: +3V3 -> GNDA
- U1 pad 17: unconnected-(U1-TXCO-Pad17) -> GNDA
- U1 pad 2: /RF/TXEN -> Net-(L2-Pad1)
- U1 pad 3: GNDA -> Net-(L2-Pad1)
- U1 pad 5: Net-(U1-RFN24) -> GNDA
- U1 pad 8: unconnected-(U1-RFP09-Pad8) -> GNDA
- U1 pad 9: unconnected-(U1-RFN09-Pad9) -> Net-(U1-SS/TR)
- U2 pad 1: Net-(J7-DP1) -> Net-(J7-DN1)
- U2 pad 3: Net-(J7-DN1) -> Net-(J7-DP1)
- U2 pad 4: /Connectors/CON_USB_D- -> /Connectors/CON_USB_D+
- U2 pad 6: /Connectors/CON_USB_D+ -> /Connectors/CON_USB_D-
- U4 pad 1: unconnected-(U4-PE2-Pad1) -> /MCU/SPI4_SCLK
- U4 pad 16: /MCU/SPI2_MOSI -> unconnected-(U4-PC1-Pad16)
- U4 pad 17: /MCU/SPI2_MISO -> unconnected-(U4-PC2_C-Pad17)
- U4 pad 18: /MCU/SPI2_CS_LCD -> unconnected-(U4-PC3_C-Pad18)
- U4 pad 29: unconnected-(U4-PA5-Pad29) -> /MCU/SPI1_SCLK
- U4 pad 30: unconnected-(U4-PA6-Pad30) -> /MCU/SPI1_MISO
- U4 pad 31: /Inputs/Slider_L -> /MCU/SPI1_MOSI
- U4 pad 32: unconnected-(U4-PC4-Pad32) -> /MCU/SPI1_CS
- U4 pad 33: unconnected-(U4-PC5-Pad33) -> /MCU/SPI1_DC
- U4 pad 34: /Inputs/Slider_R -> unconnected-(U4-PB0-Pad34)
- U4 pad 36: /MCU/SPI3_MOSI -> unconnected-(U4-PB2-Pad36)
- U4 pad 4: unconnected-(U4-PE5-Pad4) -> /MCU/SPI4_MISO
- U4 pad 40: /MCU/RF_NRST -> unconnected-(U4-PE10-Pad40)
- U4 pad 41: /MCU/SPI4_CS_RF -> unconnected-(U4-PE11-Pad41)
- U4 pad 42: /MCU/SPI4_SCLK_RF -> unconnected-(U4-PE12-Pad42)
- U4 pad 43: /MCU/SPI4_MISO_RF -> unconnected-(U4-PE13-Pad43)
- U4 pad 5: /MCU/SPI4_MOSI_RF -> /MCU/SPI4_MOSI
- U4 pad 52: /MCU/SPI2_SCLK -> unconnected-(U4-PB13-Pad52)
- U4 pad 66: unconnected-(U4-PC9-Pad66) -> /MCU/I2C3_SDA
- U4 pad 67: unconnected-(U4-PA8-Pad67) -> /MCU/I2C3_SCL
- U4 pad 78: /MCU/SPI3_SCLK -> unconnected-(U4-PC10-Pad78)
- U4 pad 79: /MCU/SPI3_MISO -> unconnected-(U4-PC11-Pad79)
- U4 pad 80: /MCU/SPI3_CS_ADC -> unconnected-(U4-PC12-Pad80)
- U8 pad 16: Net-(U8-PMID) -> VDD_LOAD_PRE_SW
Routing:
- net VDD_USB: track 0.00 -> 78.4 mm, vias 0 -> 1
- net VDD_BATT: track 0.00 -> 39.4 mm
- net VDD_LOAD: track 0.00 -> 35.8 mm
- net /MCU/SPI4_MOSI: track 0.00 -> 31.6 mm
- net /MCU/SPI4_SCLK: track 0.00 -> 30.0 mm, vias 0 -> 1
- net /MCU/I2C2_SDA: track 0.00 -> 27.7 mm, vias 0 -> 1
- net /MCU/I2C2_SCL: track 0.00 -> 25.8 mm, vias 0 -> 1
- net /MCU/I2C1_SCL: track 0.00 -> 18.8 mm, vias 0 -> 1
- net /MCU/I2C1_SDA: track 0.00 -> 17.9 mm, vias 0 -> 1
- net +3V3: track 0.00 -> 16.6 mm, vias 0 -> 2
- net /Power/REGN: track 0.00 -> 12.1 mm
- net GND_BATT: track 0.00 -> 10.4 mm
- net Net-(U10-VIN): track 0.00 -> 9.11 mm
- net Net-(J7-DP1): track 0.00 -> 6.20 mm
- net Net-(J7-DN1): track 0.00 -> 5.53 mm
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Other:
- board size 8.6 x 5 mm -> 138 x 77 mm
- board text added: "+"
- board text added: "-"
- board text added: "RF ZONE"

Commit message: Did a bunch of stuff on the controller
Parts:
- added R19: 4.7kohm, Resistor_SMD:R_0603_1608Metric, F.Cu at (166.5, 79.0)
- added R20: 4.7kohm, Resistor_SMD:R_0603_1608Metric, F.Cu at (168.1, 79.0)
- C10, C11, C12, C13, C21, C4, C5, C6, C7, C8, C9: footprint Capacitor_SMD:C_0201_0603Metric -> Capacitor_SMD:C_0603_1608Metric
- R11, R12: footprint Resistor_SMD:R_0201_0603Metric -> Capacitor_SMD:C_0603_1608Metric
- R14, R15: footprint Resistor_SMD:R_0603_1608Metric -> Capacitor_SMD:C_0603_1608Metric
- R16, R2: footprint Resistor_THT:R_Axial_DIN0309_L9.0mm_D3.2mm_P15.24mm_Horizontal -> Capacitor_SMD:C_0603_1608Metric
- R5, R6: value 10kohm -> 4.7kohm
- moved C8 109.0 mm to (160.5, 61.1)
- moved C9 103.1 mm to (160.5, 59.4)
- moved C10 102.8 mm to (144.4, 56.4)
- moved C11 101.8 mm to (174.5, 71.6)
- moved C21 101.8 mm to (176.9, 68.1)
- moved R11 101.8 mm to (176.9, 69.8)
- moved R12 101.8 mm to (176.9, 71.6)
- moved C12 99.8 mm to (139.8, 61.8), turned to 90 degrees
- moved Y1 99.6 mm to (137.7, 66.8), turned to 90 degrees
- moved C4 94.6 mm to (137.0, 61.8), turned to 90 degrees
- moved C13 94.6 mm to (140.5, 69.1), turned to 90 degrees
- moved C7 91.3 mm to (176.8, 73.2)
- moved C6 89.2 mm to (137.7, 71.0), turned to 180 degrees
- moved C5 85.9 mm to (137.7, 72.6), turned to 180 degrees
- moved D2 77.1 mm to (114.4, 95.9), turned to -90 degrees
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Connections:
- J3 pad 5: /Outputs/LCD_CS -> /MCU/SPI4_CS
- J3 pad 6: /Outputs/LCD_DC -> /MCU/SPI4_DC
- R5 pad 1: /MCU/I2C3_SCL -> /MCU/I2C1_SCL
- R6 pad 1: /MCU/I2C3_SDA -> /MCU/I2C1_SDA
- U10 pad 3: /MCU/I2C3_SDA -> /MCU/I2C1_SDA
- U10 pad 4: /MCU/I2C3_SCL -> /MCU/I2C1_SCL
- U4 pad 29: /MCU/SPI1_SCLK -> unconnected-(U4-PA5-Pad29)
- U4 pad 3: unconnected-(U4-PE4-Pad3) -> /MCU/SPI4_CS
- U4 pad 30: /MCU/SPI1_MISO -> unconnected-(U4-PA6-Pad30)
- U4 pad 31: /MCU/SPI1_MOSI -> unconnected-(U4-PA7-Pad31)
- U4 pad 32: /MCU/SPI1_CS -> unconnected-(U4-PC4-Pad32)
- U4 pad 33: /MCU/SPI1_DC -> unconnected-(U4-PC5-Pad33)
- U4 pad 4: /MCU/SPI4_MISO -> /MCU/SPI4_DC
- U4 pad 65: unconnected-(U4-PC8-Pad65) -> /MCU/SDMMC1_D0
- U4 pad 66: /MCU/I2C3_SDA -> /MCU/SDMMC1_D1
- U4 pad 67: /MCU/I2C3_SCL -> unconnected-(U4-PA8-Pad67)
- U4 pad 76: /Connectors/SWCLK -> unconnected-(U4-PA14-Pad76)
- U4 pad 77: /Connectors/SWDIO -> unconnected-(U4-PA15-Pad77)
- U4 pad 78: unconnected-(U4-PC10-Pad78) -> /MCU/SDMMC1_D2
- U4 pad 79: unconnected-(U4-PC11-Pad79) -> /MCU/SDMMC1_D3
- U4 pad 80: unconnected-(U4-PC12-Pad80) -> /MCU/SDMMC1_CK
- U4 pad 81: /Inputs/Button_L -> unconnected-(U4-PD0-Pad81)
- U4 pad 82: /Inputs/Button_R -> unconnected-(U4-PD1-Pad82)
- U4 pad 83: unconnected-(U4-PD2-Pad83) -> /MCU/SDMMC1_CMD
Routing:
- net +3V3: track 16.6 -> 180.7 mm
- net /MCU/I2C1_SDA: track 17.9 -> 52.4 mm, vias 1 -> 0
- net VDD_USB: track 78.4 -> 111.8 mm, vias 1 -> 2
- net /MCU/I2C1_SCL: track 18.8 -> 50.4 mm, vias 1 -> 0
- net VDD_LOAD_PRE_SW: track 4.23 -> 34.9 mm, vias 0 -> 7
- net /MCU/SPI4_DC: track 0.00 -> 27.2 mm, vias 0 -> 2
- net /MCU/SDMMC1_CMD: track 0.00 -> 25.2 mm
- net /MCU/I2C2_SDA: track 27.7 -> 2.74 mm, vias 1 -> 0
- net /MCU/SPI4_CS: track 0.00 -> 24.3 mm, vias 0 -> 2
- net /MCU/SDMMC1_CK: track 0.00 -> 23.5 mm
- net /MCU/I2C2_SCL: track 25.8 -> 2.73 mm, vias 1 -> 0
- net GNDA: track 2.06 -> 24.9 mm, vias 23 -> 44
- net /MCU/SDMMC1_D3: track 0.00 -> 22.7 mm
- net /MCU/SDMMC1_D2: track 0.00 -> 22.0 mm
- net /MCU/SDMMC1_D0: track 0.00 -> 16.5 mm
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