File: RC-Car-Controller/Outputs.kicad_sch (KiCad schematic)
At the start: 3 parts, among them J3 Conn_01x08_Pin

Commit message: Did some stuff on the Controller
Parts:
- J3: footprint Connector_PinHeader_2.54mm:PinHeader_1x08_P2.54mm_Vertical -> 2inch_LCD:2inch_LCD
Changed lines of the file:
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@@
 			)
 		)
-		(property "Footprint" "Connector_PinHeader_2.54mm:PinHeader_1x08_P2.54mm_Vertical"
+		(property "Footprint" "2inch_LCD:2inch_LCD"
 			(at 86.36 90.17 0)
 			(effects

Commit message: Finished Controller PCB Pre-Review
Parts:
- renumbered J3 to J6
Changed lines of the file:
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@@
 		(on_board yes)
 		(dnp no)
-		(property "Reference" "#PWR025"
+		(property "Reference" "#PWR096"
 			(at 97.79 85.09 0)
 			(effects
@@
 			(project "RC-Car-Controller"
 				(path "/ba870fd1-751d-4755-8e1a-1ea86ca9e2f6/c7631c9a-9d0f-4b64-bf26-f76b69ba0d74"
-					(reference "#PWR025")
+					(reference "#PWR096")
 					(unit 1)
 				)
@@
 		(on_board yes)
 		(dnp no)
-		(property "Reference" "#PWR022"
+		(property "Reference" "#PWR095"
 			(at 87.63 82.55 0)
 			(effects
@@
 			(project "RC-Car-Controller"
 				(path "/ba870fd1-751d-4755-8e1a-1ea86ca9e2f6/c7631c9a-9d0f-4b64-bf26-f76b69ba0d74"
-					(reference "#PWR022")
+					(reference "#PWR095")
 					(unit 1)
 				)
@@
 		(on_board yes)
 		(dnp no)
-		(property "Reference" "J3"
+		(property "Reference" "J6"
 			(at 80.264 91.186 0)
 			(effects
@@
 			(project ""
 				(path "/ba870fd1-751d-4755-8e1a-1ea86ca9e2f6/c7631c9a-9d0f-4b64-bf26-f76b69ba0d74"
-					(reference "J3")
+					(reference "J6")
 					(unit 1)
 				)
@@
 		(on_board yes)
 		(dnp no)
-		(property "Reference" "#PWR026"
+		(property "Reference" "#PWR097"
 			(at 87.63 100.33 0)
 			(effects
@@
 			(project "RC-Car-Controller"
 				(path "/ba870fd1-751d-4755-8e1a-1ea86ca9e2f6/c7631c9a-9d0f-4b64-bf26-f76b69ba0d74"
-					(reference "#PWR026")
+					(reference "#PWR097")
 					(unit 1)
 				)
@@
 		(on_board yes)
 		(dnp no)
-		(property "Reference" "#PWR027"
+		(property "Reference" "#PWR0100"
 			(at 134.62 100.33 0)
 			(effects
@@
 			(project "RC-Car-Controller"
 				(path "/ba870fd1-751d-4755-8e1a-1ea86ca9e2f6/c7631c9a-9d0f-4b64-bf26-f76b69ba0d74"
-					(reference "#PWR027")
+					(reference "#PWR0100")
 					(unit 1)
 				)
@@
 		(on_board yes)
 		(dnp no)
-		(property "Reference" "#PWR024"
+		(property "Reference" "#PWR099"
 			(at 124.46 87.63 0)
 			(effects
@@
 			(project "RC-Car-Controller"
 				(path "/ba870fd1-751d-4755-8e1a-1ea86ca9e2f6/c7631c9a-9d0f-4b64-bf26-f76b69ba0d74"
-					(reference "#PWR024")
+					(reference "#PWR099")
 					(unit 1)
 				)
@@
 		(on_board yes)
 		(dnp no)
-		(property "Reference" "#PWR028"
+		(property "Reference" "#PWR0101"
 			(at 124.46 102.87 0)
 			(effects
@@
 			(project "RC-Car-Controller"
 				(path "/ba870fd1-751d-4755-8e1a-1ea86ca9e2f6/c7631c9a-9d0f-4b64-bf26-f76b69ba0d74"
-					(reference "#PWR028")
+					(reference "#PWR0101")
 					(unit 1)
 				)
@@
 		(on_board yes)
 		(dnp no)
-		(property "Reference" "#PWR023"
+		(property "Reference" "#PWR098"
 			(at 134.62 85.09 0)
 			(effects
@@
 			(project "RC-Car-Controller"
 				(path "/ba870fd1-751d-4755-8e1a-1ea86ca9e2f6/c7631c9a-9d0f-4b64-bf26-f76b69ba0d74"
-					(reference "#PWR023")
-					(unit 1)
-				)
+					(reference "#PWR098")
+					(unit 1)
+				)

Commit message: Filled out some Controller Caps
Parts:
- Brd1, Brd2, J6: MANUF_PN (none) -> N/A
Changed lines of the file:
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@@
 			)
 		)
-		(property "MANUF_PN" ""
+		(property "MANUF_PN" "N/A"
 			(at 86.36 90.17 0)
 			(effects
@@
 			)
 		)
-		(property "MANUF_PN" ""
+		(property "MANUF_PN" "N/A"
 			(at 139.7 99.06 0)
 			(effects
@@
 			)
 		)
-		(property "MANUF_PN" ""
+		(property "MANUF_PN" "N/A"
 			(at 139.7 83.82 0)
 			(effects
