File: RC-Car-Controller/RF_sch.kicad_sch (KiCad schematic)
At the start: 34 parts

Commit message: Added Schem PNs
Parts:
- C23, C27: MANUF_PN (none) -> CL10A106KP8NNNC
Changed lines of the file:
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@@
 			)
 		)
-		(property "MANUF_PN" ""
+		(property "MANUF_PN" "CL10A106KP8NNNC"
 			(at 207.01 35.56 0)
 			(effects
@@
 			)
 		)
-		(property "MANUF_PN" ""
+		(property "MANUF_PN" "CL10A106KP8NNNC"
 			(at 160.02 35.56 0)
 			(effects
