File: RC-Car-Controller/MCU_sch.kicad_sch (KiCad schematic)
At the start: 22 parts, among them SW1 SW_Push, SW3 SW_SPDT, U4 STM32H743VGTx, Y1 Crystal

Commit message: Finished Controller PCB Pre-Review
Parts:
- renumbered C4 to C12, C5 to C13, C6 to C14, C7 to C15, C8 to C16, C9 to C17, C10 to C18, C11 to C19, C12 to C20, C13 to C21, C21 to C22, R11 to R16, R12 to R17, R25 to R18, R5 to R19, R6 to R20, R19 to R21, R20 to R22, SW3 to SW2, U4 to U5
Connections:
- net RF_RESET: now also U5.81 (PD0)
- net SWDIO: now also U5.72 (PA13); no longer U5.77 (PA15)
- no-connect marks 55 -> 54

Commit message: Fixed GPIOADC
Connections:
- net BTN_L: now also U5.29 (PA5); no longer U5.30 (PA6)
- net WIPE_L: now also U5.30 (PA6); no longer U5.31 (PA7)
Changed lines of the file:
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@@
+	)
+	(no_connect
+		(at 143.51 60.96)
 	)
 	(no_connect
@@
 	(no_connect
 		(at 143.51 50.8)
-	)
-	(no_connect
-		(at 143.51 55.88)
 	)
 	(no_connect
@@
 	(hierarchical_label "BTN_L"
 		(shape input)
+		(at 143.51 55.88 0)
+		(fields_autoplaced yes)
+		(effects
+			(font
+				(size 1.27 1.27)
+			)
+			(justify left)
+		)
+	)
+	(hierarchical_label "SDMMC1_CK"
+		(shape input)
+		(at 143.51 160.02 0)
+		(fields_autoplaced yes)
+		(effects
+			(font
+				(size 1.27 1.27)
+			)
+			(justify left)
+		)
+	)
+	(hierarchical_label "I2C1_SDA"
+		(shape input)
+		(at 143.51 109.22 0)
+		(fields_autoplaced yes)
+		(effects
+			(font
+				(size 1.27 1.27)
+			)
+			(justify left)
+		)
+	)
+	(hierarchical_label "SDMMC1_D0"
+		(shape input)
+		(at 143.51 149.86 0)
+		(fields_autoplaced yes)
+		(effects
+			(font
+				(size 1.27 1.27)
+			)
+			(justify left)
+		)
+	)
+	(hierarchical_label "SDMMC1_CMD"
+		(shape input)
+		(at 97.79 114.3 180)
+		(fields_autoplaced yes)
+		(effects
+			(font
+				(size 1.27 1.27)
+			)
+			(justify right)
+		)
+	)
+	(hierarchical_label "SWDIO"
+		(shape input)
+		(at 143.51 76.2 0)
+		(fields_autoplaced yes)
+		(effects
+			(font
+				(size 1.27 1.27)
+			)
+			(justify left)
+		)
+	)
+	(hierarchical_label "I2C2_SCL"
+		(shape input)
+		(at 143.51 111.76 0)
+		(fields_autoplaced yes)
+		(effects
+			(font
+				(size 1.27 1.27)
+			)
+			(justify left)
+		)
+	)
+	(hierarchical_label "BTN_R"
+		(shape input)
+		(at 143.51 142.24 0)
+		(fields_autoplaced yes)
+		(effects
+			(font
+				(size 1.27 1.27)
+			)
+			(justify left)
+		)
+	)
+	(hierarchical_label "MCU_USB_D+"
+		(shape input)
+		(at 143.51 73.66 0)
+		(fields_autoplaced yes)
+		(effects
+			(font
+				(size 1.27 1.27)
+			)
+			(justify left)
+		)
+	)
+	(hierarchical_label "I2C2_SDA"
+		(shape input)
+		(at 208.28 85.09 270)
+		(fields_autoplaced yes)
+		(effects
+			(font
+				(size 1.27 1.27)
+			)
+			(justify right)
+		)
+	)
+	(hierarchical_label "I2C2_SCL"
+		(shape input)
+		(at 205.74 85.09 270)
+		(fields_autoplaced yes)
+		(effects
+			(font
+				(size 1.27 1.27)
+			)
+			(justify right)
+		)
+	)
+	(hierarchical_label "NRST"
+		(shape input)
+		(at 97.79 43.18 180)
+		(fields_autoplaced yes)
+		(effects
+			(font
+				(size 1.27 1.27)
+			)
+			(justify right)
+		)
+	)
+	(hierarchical_label "SDMMC1_D1"
+		(shape input)
+		(at 143.51 152.4 0)
+		(fields_autoplaced yes)
+		(effects
+			(font
+				(size 1.27 1.27)
+			)
+			(justify left)
+		)
+	)
+	(hierarchical_label "NRST"
+		(shape input)
+		(at 53.34 100.33 0)
+		(fields_autoplaced yes)
+		(effects
+			(font
+				(size 1.27 1.27)
+			)
+			(justify left)
+		)
+	)
+	(hierarchical_label "WIPE_L"
+		(shape input)
 		(at 143.51 58.42 0)
 		(fields_autoplaced yes)
 		(effects
-			(font
-				(size 1.27 1.27)
-			)
-			(justify left)
-		)
-	)
-	(hierarchical_label "SDMMC1_CK"
-		(shape input)
-		(at 143.51 160.02 0)
-		(fields_autoplaced yes)
-		(effects
-			(font
-				(size 1.27 1.27)
-			)
-			(justify left)
-		)
-	)
-	(hierarchical_label "I2C1_SDA"
-		(shape input)
-		(at 143.51 109.22 0)
-		(fields_autoplaced yes)
-		(effects
-			(font
-				(size 1.27 1.27)
-			)
-			(justify left)
-		)
-	)
-	(hierarchical_label "SDMMC1_D0"
-		(shape input)
-		(at 143.51 149.86 0)
-		(fields_autoplaced yes)
-		(effects
-			(font
-				(size 1.27 1.27)
-			)
-			(justify left)
-		)
-	)
-	(hierarchical_label "SDMMC1_CMD"
-		(shape input)
-		(at 97.79 114.3 180)
-		(fields_autoplaced yes)
-		(effects
-			(font
-				(size 1.27 1.27)
-			)
-			(justify right)
-		)
-	)
-	(hierarchical_label "SWDIO"
-		(shape input)
-		(at 143.51 76.2 0)
-		(fields_autoplaced yes)
-		(effects
-			(font
-				(size 1.27 1.27)
-			)
-			(justify left)
-		)
-	)
-	(hierarchical_label "I2C2_SCL"
-		(shape input)
-		(at 143.51 111.76 0)
-		(fields_autoplaced yes)
-		(effects
-			(font
-				(size 1.27 1.27)
-			)
-			(justify left)
-		)
-	)
-	(hierarchical_label "BTN_R"
-		(shape input)
-		(at 143.51 142.24 0)
-		(fields_autoplaced yes)
-		(effects
-			(font
-				(size 1.27 1.27)
-			)
-			(justify left)
-		)
-	)
-	(hierarchical_label "MCU_USB_D+"
-		(shape input)
-		(at 143.51 73.66 0)
-		(fields_autoplaced yes)
-		(effects
-			(font
-				(size 1.27 1.27)
-			)
-			(justify left)
-		)
-	)
-	(hierarchical_label "I2C2_SDA"
-		(shape input)
-		(at 208.28 85.09 270)
-		(fields_autoplaced yes)
-		(effects
-			(font
-				(size 1.27 1.27)
-			)
-			(justify right)
-		)
-	)
-	(hierarchical_label "I2C2_SCL"
-		(shape input)
-		(at 205.74 85.09 270)
-		(fields_autoplaced yes)
-		(effects
-			(font
-				(size 1.27 1.27)
-			)
-			(justify right)
-		)
-	)
-	(hierarchical_label "NRST"
-		(shape input)
-		(at 97.79 43.18 180)
-		(fields_autoplaced yes)
-		(effects
-			(font
-				(size 1.27 1.27)
-			)
-			(justify right)
-		)
-	)
-	(hierarchical_label "SDMMC1_D1"
-		(shape input)
-		(at 143.51 152.4 0)
-		(fields_autoplaced yes)
-		(effects
-			(font
-				(size 1.27 1.27)
-			)
-			(justify left)
-		)
-	)
-	(hierarchical_label "NRST"
-		(shape input)
-		(at 53.34 100.33 0)
-		(fields_autoplaced yes)
-		(effects
-			(font
-				(size 1.27 1.27)
-			)
-			(justify left)
-		)
-	)
-	(hierarchical_label "WIPE_L"
-		(shape input)
-		(at 143.51 60.96 0)
-		(fields_autoplaced yes)
-		(effects

Commit message: most resistors given PNs
most resistors given PNs. some remaining
Parts:
- R16, R17, R18: MANUF_PN (none) -> RC0603FR-0710KL
Changed lines of the file:
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@@
+			)
+		)
+		(property "MANUF_PN" ""
+			(at 177.8 36.83 0)
+			(effects
+				(font
+					(size 1.27 1.27)
+				)
+				(hide yes)
 			)
 		)
@@
 			)
 		)
+		(property "MANUF_PN" ""
+			(at 195.58 36.83 0)
+			(effects
+				(font
+					(size 1.27 1.27)
+				)
+				(hide yes)
+			)
+		)
 		(pin "1"
 		)
@@
 			)
 		)
+		(property "MANUF_PN" "RC0603FR-0710KL"
+			(at 48.26 96.52 0)
+			(effects
+				(font
+					(size 1.27 1.27)
+				)
+				(hide yes)
+			)
+		)
 		(pin "2"
 		)
@@
 			)
 		)
+		(property "MANUF_PN" ""
+			(at 232.41 81.28 0)
+			(effects
+				(font
+					(size 1.27 1.27)
+				)
+				(hide yes)
+			)
+		)
 		(pin "1"
 		)
@@
 			)
 		)
+		(property "MANUF_PN" ""
+			(at 59.69 62.23 0)
+			(effects
+				(font
+					(size 1.27 1.27)
+				)
+				(hide yes)
+			)
+		)
 		(pin "1"
 		)
@@
 			)
 		)
+		(property "MANUF_PN" ""
+			(at 208.28 81.28 0)
+			(effects
+				(font
+					(size 1.27 1.27)
+				)
+				(hide yes)
+			)
+		)
 		(pin "1"
 		)
@@
 			)
 		)
+		(property "MANUF_PN" "RC0603FR-0710KL"
+			(at 74.93 45.72 0)
+			(effects
+				(font
+					(size 1.27 1.27)
+				)
+				(hide yes)
+			)
+		)
 		(pin "2"
 		)
@@
 			)
 		)
+		(property "MANUF_PN" ""
+			(at 248.92 36.83 0)
+			(effects
+				(font
+					(size 1.27 1.27)
+				)
+				(hide yes)
+			)
+		)
 		(pin "1"
 		)
@@
 			)
 		)
+		(property "MANUF_PN" ""
+			(at 205.74 81.28 0)
+			(effects
+				(font
+					(size 1.27 1.27)
+				)
+				(hide yes)
+			)
+		)
 		(pin "1"
 		)
@@
 			)
 		)
+		(property "MANUF_PN" ""
+			(at 83.82 48.26 0)
+			(effects
+				(font
+					(size 1.27 1.27)
+				)
+				(hide yes)
+			)
+		)
 		(pin "2"
 		)
@@
 			)
 		)
+		(property "MANUF_PN" ""
+			(at 229.87 81.28 0)
+			(effects
+				(font
+					(size 1.27 1.27)
+				)
+				(hide yes)
+			)
+		)
 		(pin "1"
 		)
@@
 			)
 		)
+		(property "MANUF_PN" ""
+			(at 69.85 160.02 0)
+			(effects
+				(font
+					(size 1.27 1.27)
+				)
+				(hide yes)
+			)
+		)
 		(pin "1"
 		)
@@
 			)
 		)
+		(property "MANUF_PN" ""
+			(at 87.63 160.02 0)
+			(effects
+				(font
+					(size 1.27 1.27)
+				)
+				(hide yes)
+			)
+		)
 		(pin "1"
 		)
@@
 			)
 		)
+		(property "MANUF_PN" ""
+			(at 48.26 104.14 0)
+			(effects
+				(font
+					(size 1.27 1.27)
+				)
+				(hide yes)
+			)
+		)
 		(pin "1"
 		)
@@
 			)
 		)
+		(property "MANUF_PN" ""
+			(at 231.14 36.83 0)
+			(effects
+				(font
+					(size 1.27 1.27)
+				)
+				(hide yes)
+			)
+		)
 		(pin "1"
 		)
@@
 			)
 		)
+		(property "MANUF_PN" ""
+			(at 50.8 58.42 0)
+			(effects
+				(font
+					(size 1.27 1.27)
+				)
+				(hide yes)
+			)
+		)
 		(pin "2"
 		)
@@
 			)
 		)
+		(property "MANUF_PN" ""
+			(at 40.64 62.23 0)
+			(effects
+				(font
+					(size 1.27 1.27)
+				)
+				(hide yes)
+			)
+		)
 		(pin "1"
 		)
@@
 			)
 		)
+		(property "MANUF_PN" ""
+			(at 120.65 106.68 0)
+			(effects
+				(font
+					(size 1.27 1.27)
+				)
+				(hide yes)
+			)
+		)
 		(pin "38"
 		)
@@
 			)
 		)
+		(property "MANUF_PN" "RC0603FR-0710KL"
+			(at 74.93 50.8 0)
+			(effects
+				(font
+					(size 1.27 1.27)
+				)
+				(hide yes)
+			)
+		)
 		(pin "2"
 		)
@@
 			)
 		)
+		(property "MANUF_PN" ""
+			(at 160.02 36.83 0)
+			(effects
+				(font
+					(size 1.27 1.27)
+				)
+				(hide yes)
+			)
+		)
 		(pin "1"
 		)
@@
 			)
 		)
+		(property "MANUF_PN" ""
+			(at 213.36 36.83 0)
+			(effects
+				(font
+					(size 1.27 1.27)
+				)
+				(hide yes)
+			)
+		)
 		(pin "1"
 		)
@@
 			(at 40.64 100.33 0)
 			(effects
+				(font
+					(size 1.27 1.27)
+				)
+				(hide yes)
+			)
+		)
+		(property "MANUF_PN" ""
+			(at 40.64 100.33 0)
+			(effects

Commit message: controller cpnts given MANUF_PNs
controller cpnts given MANUF_PNs. not all components, but all resistors are done
Parts:
- R19, R20, R21, R22: MANUF_PN (none) -> ERA-3ARW472V
Changed lines of the file:
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@@
 			)
 		)
-		(property "MANUF_PN" ""
+		(property "MANUF_PN" "ERA-3ARW472V"
 			(at 232.41 81.28 0)
 			(effects
@@
 			)
 		)
-		(property "MANUF_PN" ""
+		(property "MANUF_PN" "ERA-3ARW472V"
 			(at 208.28 81.28 0)
 			(effects
@@
 			)
 		)
-		(property "MANUF_PN" ""
+		(property "MANUF_PN" "ERA-3ARW472V"
 			(at 205.74 81.28 0)
 			(effects
@@
 			)
 		)
-		(property "MANUF_PN" ""
+		(property "MANUF_PN" "ERA-3ARW472V"
 			(at 229.87 81.28 0)
 			(effects

Commit message: Filled out some Controller Caps
Parts:
- C12, C13, C14: MANUF_PN (none) -> C0603C180J5GACTU
- C15, C16: MANUF_PN (none) -> C0603C225K4PACTU
- C17, C18, C19, C20, C21, C22: MANUF_PN (none) -> C0603C104K5RAC7411
- SW2: MANUF_PN (none) -> N/A
- U5: MANUF_PN (none) -> STM32H743VGT6
Changed lines of the file:
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@@
 			)
 		)
-		(property "MANUF_PN" ""
+		(property "MANUF_PN" "C0603C104K5RAC7411"
 			(at 177.8 36.83 0)
 			(effects
@@
 			)
 		)
-		(property "MANUF_PN" ""
+		(property "MANUF_PN" "C0603C104K5RAC7411"
 			(at 195.58 36.83 0)
 			(effects
@@
 			)
 		)
-		(property "MANUF_PN" ""
+		(property "MANUF_PN" "C0603C180J5GACTU"
 			(at 59.69 62.23 0)
 			(effects
@@
 			)
 		)
-		(property "MANUF_PN" ""
+		(property "MANUF_PN" "C0603C104K5RAC7411"
 			(at 248.92 36.83 0)
 			(effects
@@
 			)
 		)
-		(property "MANUF_PN" ""
+		(property "MANUF_PN" "N/A"
 			(at 83.82 48.26 0)
 			(effects
@@
 			)
 		)
-		(property "MANUF_PN" ""
+		(property "MANUF_PN" "C0603C225K4PACTU"
 			(at 69.85 160.02 0)
 			(effects
@@
 			)
 		)
-		(property "MANUF_PN" ""
+		(property "MANUF_PN" "C0603C225K4PACTU"
 			(at 87.63 160.02 0)
 			(effects
@@
 			)
 		)
-		(property "MANUF_PN" ""
+		(property "MANUF_PN" "C0603C180J5GACTU"
 			(at 48.26 104.14 0)
 			(effects
@@
 			)
 		)
-		(property "MANUF_PN" ""
+		(property "MANUF_PN" "C0603C104K5RAC7411"
 			(at 231.14 36.83 0)
 			(effects
@@
 			)
 		)
-		(property "MANUF_PN" ""
+		(property "MANUF_PN" "C0603C180J5GACTU"
 			(at 40.64 62.23 0)
 			(effects
@@
 			)
 		)
-		(property "MANUF_PN" ""
+		(property "MANUF_PN" "STM32H743VGT6"
 			(at 120.65 106.68 0)
 			(effects
@@
 			)
 		)
-		(property "MANUF_PN" ""
+		(property "MANUF_PN" "C0603C104K5RAC7411"
 			(at 160.02 36.83 0)
 			(effects
@@
 			)
 		)
-		(property "MANUF_PN" ""
+		(property "MANUF_PN" "C0603C104K5RAC7411"
 			(at 213.36 36.83 0)
 			(effects

Commit message: Added Schem PNs
Parts:
- Y1: MANUF_PN (none) -> ABM7-25.000MHZ-D2Y-T
Changed lines of the file:
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@@
 			)
 		)
-		(property "MANUF_PN" ""
+		(property "MANUF_PN" "ABM7-25.000MHZ-D2Y-T"
 			(at 50.8 58.42 0)
 			(effects

Commit message: Finished BOM Drafts
Parts:
- SW1: MANUF_PN (none) -> 1825910-6
Changed lines of the file:
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@@
 			)
 		)
-		(property "MANUF_PN" ""
+		(property "MANUF_PN" "1825910-6"
 			(at 40.64 100.33 0)
 			(effects
