File: RC-Car-Controller/RC-Car-Controller.kicad_sch (KiCad schematic)
At the start: 12 parts

Commit message: Filled out some Controller Caps
Parts:
- TP1, TP2, TP3, TP4, TP5, TP6: MANUF_PN (none) -> N/A
Changed lines of the file:
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@@
 			)
 		)
-		(property "MANUF_PN" ""
+		(property "MANUF_PN" "N/A"
 			(at 238.149 31.1872 0)
 			(effects
@@
 			)
 		)
-		(property "MANUF_PN" ""
+		(property "MANUF_PN" "N/A"
 			(at 238.149 45.1572 0)
 			(effects
@@
 			)
 		)
-		(property "MANUF_PN" ""
+		(property "MANUF_PN" "N/A"
 			(at 227.989 45.1572 0)
 			(effects
@@
 			)
 		)
-		(property "MANUF_PN" ""
+		(property "MANUF_PN" "N/A"
 			(at 249.579 31.1872 0)
 			(effects
@@
 			)
 		)
-		(property "MANUF_PN" ""
+		(property "MANUF_PN" "N/A"
 			(at 227.989 31.1872 0)
 			(effects
@@
 			)
 		)
-		(property "MANUF_PN" ""
+		(property "MANUF_PN" "N/A"
 			(at 249.579 45.1572 0)
 			(effects

Commit message: Finished BOM Drafts
Parts:
- D1, D2: MANUF_PN (none) -> LTST-C190GKT
- D3: MANUF_PN (none) -> LTL-4293
- R3: value 60ohm -> 220ohm; MANUF_PN RMCF0603FT62R0 -> RMCF0603FT220R
Changed lines of the file:
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@@
 			)
 		)
-		(property "MANUF_PN" ""
+		(property "MANUF_PN" "LTST-C190GKT"
 			(at 180.34 41.91 0)
 			(effects
@@
 			)
 		)
-		(property "Value" "60ohm"
+		(property "Value" "220ohm"
 			(at 198.12 35.5599 0)
 			(effects
@@
 			)
 		)
-		(property "MANUF_PN" "RMCF0603FT62R0"
+		(property "MANUF_PN" "RMCF0603FT220R"
 			(at 195.58 34.29 0)
 			(effects
@@
 			)
 		)
-		(property "MANUF_PN" ""
+		(property "MANUF_PN" "LTST-C190GKT"
 			(at 166.37 41.91 0)
 			(effects
@@
 			)
 		)
-		(property "MANUF_PN" ""
+		(property "MANUF_PN" "LTL-4293"
 			(at 195.58 41.91 0)
 			(effects
